File: hardware/odeck-10/mcu.kicad_sch (KiCad schematic)
At the start: 0 parts

Commit message: Draft remaining sheets: USB-A, card reader, Ethernet, MCU, display/UI, sensors
- usb_a: 2x 10G USB-A, TPS2553 switches (hub OR RP2350 force), INA180 sense
- card_reader: GL3224 + SD/microSD, card detect + activity to MCU
- ethernet: RTL8156BG with switched 3.3 V, 0.95 V PWM buck, 2.5G magjack,
  LED buffer, EUI-48 EEPROM + gated I2C bridge for MAC eFuse write
- mcu: RP2350B reference core, full GPIO table, TCA9534 expander, PIO I2C
- display_ui: 2.0" ST7789 LCD + backlight PWM, buttons, unpopulated GPIO
  header (series R + ESD), Qwiic
- sensors: 8x TMP1075, 2 NTCs, thermocouple pads
- integration: ETH_I2C_EN net, TPS62933F for +3V3, PWR_FLAGs
- schgen: deterministic UUIDs; bom_check: cost summary
- 181 parts, all JLC stock >= 5; netlist verify OK; ERC clean but 1 spare pin

Co-Authored-By: Claude Opus 5.5 <noreply@anthropic.com>
Parts:
- added C1001, C1002, C1003, C1004: 4.7u, Capacitor_SMD:C_0402_1005Metric, symbol Device:C
- added C1005, C1007, C1008, C1009, C1010, C1011, C1012, C1013, C1014, C1015, C1016, C1017, C1018, C1019, C1022, C1023, C1026, C1027: 100n, Capacitor_SMD:C_0402_1005Metric, symbol Device:C
- added C1006: 10u, Capacitor_SMD:C_0603_1608Metric, symbol Device:C
- added C1020, C1021: 15p, Capacitor_SMD:C_0402_1005Metric, symbol Device:C
- added C1024, C1025: 10n, Capacitor_SMD:C_0402_1005Metric, symbol Device:C
- added D1001: PWR green, LED_SMD:LED_0805_2012Metric, symbol Device:LED
- added D1002: STATUS red, LED_SMD:LED_0603_1608Metric, symbol Device:LED
- added J1001: DEBUG UART, Connector_PinHeader_2.54mm:PinHeader_1x03_P2.54mm_Vertical, symbol Connector_Generic:Conn_01x03
- added L1001: 3.3u, odeck:IND-SMD_L2.0-W1.6_AOTA-B201610S3R3-101-T, symbol odeck:AOTA-B201610S3R3-101-T
- added R1001, R1022, R1023: 33, Resistor_SMD:R_0402_1005Metric, symbol Device:R
- added R1002: 10, Resistor_SMD:R_0402_1005Metric, symbol Device:R
- added R1003, R1005, R1006, R1025: 1k, Resistor_SMD:R_0402_1005Metric, symbol Device:R
- added R1004, R1015, R1016, R1017, R1018, R1019, R1020, R1021: 10k, Resistor_SMD:R_0402_1005Metric, symbol Device:R
- added R1007, R1008: 27, Resistor_SMD:R_0402_1005Metric, symbol Device:R
- added R1009, R1010, R1011, R1012: 2.2k, Resistor_SMD:R_0402_1005Metric, symbol Device:R
- added R1013, R1014: 4.7k, Resistor_SMD:R_0402_1005Metric, symbol Device:R
- added R1024: 330, Resistor_SMD:R_0402_1005Metric, symbol Device:R
- added SW1001: BOOTSEL, odeck:SW-SMD_4P-L5.1-W5.1-P3.70-LS6.5-TL_H1.5, symbol odeck:TS-1187A-B-A-B
- added SW1002: RESET, odeck:SW-SMD_4P-L5.1-W5.1-P3.70-LS6.5-TL_H1.5, symbol odeck:TS-1187A-B-A-B
- added TP1001: SWCLK, TestPoint:TestPoint_Pad_D1.0mm, symbol Connector:TestPoint
- added TP1002: SWDIO, TestPoint:TestPoint_Pad_D1.0mm, symbol Connector:TestPoint
- added TP1003: RUN, TestPoint:TestPoint_Pad_D1.0mm, symbol Connector:TestPoint
- added TP1004: GND, TestPoint:TestPoint_Pad_D1.0mm, symbol Connector:TestPoint
- added U1001: RP2350B, odeck:QFN-80_L10.0-W10.0-P0.40-TL-EP3.4, symbol odeck:RP2350B_C42415655
- added U1002: W25Q128JVSIQ, odeck:SOIC-8_L5.3-W5.3-P1.27-LS8.0-BL, symbol odeck:W25Q128JVSIQTR
- added U1003: TCA9534PWR, odeck:TSSOP-16_L5.0-W4.4-P0.65-LS6.4-BL, symbol odeck:TCA9534PWR
- added Y1001: 12MHz, Crystal:Crystal_SMD_3225-4Pin_3.2x2.5mm, symbol Device:Crystal_GND24
Connections:
- new net +1V1: C1002.1, C1017.1, C1018.1, C1019.1, L1001.2, U1001.10 (DVDD), U1001.32 (DVDD), U1001.51 (DVDD), U1001.65 (VREG_FB)
- new net +3V3: C1001.1, C1006.1, C1007.1, C1008.1, C1009.1, C1010.1, C1011.1, C1012.1, C1013.1, C1014.1, C1015.1, C1016.1, C1022.1, C1023.1, R1001.1, R1002.1, R1004.2, R1009.2, R1010.2, R1011.2, R1012.2, R1013.2, R1014.2, R1015.2, R1016.2, R1017.2, R1024.1, U1001.15 (IOVDD), U1001.24 (IOVDD), U1001.29 (IOVDD), U1001.41 (IOVDD), U1001.5 (IOVDD), U1001.50 (IOVDD), U1001.60 (IOVDD), U1001.64 (VREG_VIN), U1001.68 (USB_OTP_VDD), U1001.69 (QSPI_IOVDD), U1001.76 (IOVDD), U1002.8 (VCC), U1003.16 (VCC)
- new net ADC_AVDD: C1004.1, C1005.1, R1002.2, R1020.1, R1021.1, U1001.59 (ADC_AVDD)
- new net ADC_ISNS1: C1024.1, R1018.2, U1001.49 (GPIO40_ADC0)
- new net ADC_ISNS2: C1025.1, R1019.2, U1001.52 (GPIO41_ADC1)
- new net BOOTSEL_SW: R1005.2, SW1001.1 (A), SW1001.2 (B)
- new net BTN_A_N: U1001.40 (GPIO32)
- new net BTN_B_N: U1001.42 (GPIO33)
- new net CR_CD_SD_N: U1003.7 (P3)
- new net CR_CD_USD_N: U1003.9 (P4)
- new net CR_LED: U1001.48 (GPIO39)
- new net ETH_I2C_EN: U1003.11 (P6)
- new net ETH_LED0: U1001.45 (GPIO36)
- new net ETH_LED1: U1001.46 (GPIO37)
- new net ETH_LED2: U1001.47 (GPIO38)
- new net ETH_RESET_N: R1017.1, U1003.10 (P5)
- new net EXT_PWR_PRESENT: U1003.4 (P0)
- new net GND: C1001.2, C1002.2, C1003.2, C1004.2, C1005.2, C1006.2, C1007.2, C1008.2, C1009.2, C1010.2, C1011.2, C1012.2, C1013.2, C1014.2, C1015.2, C1016.2, C1017.2, C1018.2, C1019.2, C1020.2, C1021.2, C1022.2, C1023.2, C1024.2, C1025.2, C1026.2, C1027.2, D1001.1 (K), D1002.1 (K), J1001.3 (Pin_3), SW1001.3 (C), SW1001.4 (D), SW1002.3 (C), SW1002.4 (D), TP1004.1, U1001.62 (VREG_PGND), U1001.81 (GND), U1002.4 (GND), U1003.1 (A0), U1003.2 (A1), U1003.3 (A2), U1003.8 (GND), Y1001.2 (G), Y1001.4 (G)
- new net HDR_ADC0: U1001.55 (GPIO44_ADC4)
- new net HDR_ADC1: U1001.56 (GPIO45_ADC5)
- new net HDR_GPIO0: U1001.11 (GPIO12)
- new net HDR_GPIO1: U1001.12 (GPIO13)
- new net HDR_GPIO2: U1001.13 (GPIO14)
- new net HDR_GPIO3: U1001.14 (GPIO15)
- new net HDR_GPIO4: U1001.16 (GPIO16)
- new net HDR_GPIO5: U1001.17 (GPIO17)
- new net HDR_GPIO6: U1001.18 (GPIO18)
- new net HDR_GPIO7: U1001.19 (GPIO19)
- new net HUB_RESET_N: U1001.9 (GPIO11)
- new net HUB_SMB_CLK: U1001.7 (GPIO9)
- new net HUB_SMB_DAT: U1001.6 (GPIO8)
- new net HUB_SMB_PU: U1001.8 (GPIO10)
- new net I2C_EXT_SCL: R1014.1, U1001.39 (GPIO31)
- new net I2C_EXT_SDA: R1013.1, U1001.38 (GPIO30)
- new net I2C_PD_INT_N: U1001.3 (GPIO6)
- new net I2C_PD_SCL: R1012.1, U1001.2 (GPIO5)
- new net I2C_PD_SDA: R1011.1, U1001.1 (GPIO4)
- new net I2C_SYS_SCL: R1010.1, U1001.80 (GPIO3), U1003.14 (SCL)
- new net I2C_SYS_SDA: R1009.1, U1001.79 (GPIO2), U1003.15 (SDA)
- new net IOX_INT_N: R1015.1, U1001.57 (GPIO46_ADC6), U1003.13 (~{INT})
- new net IOX_P7: U1003.12 (P7)
- new net LAPTOP_OVP_N: U1003.5 (P1)
- new net LCD_BL_PWM: U1001.26 (GPIO25)
- new net LCD_CS_N: U1001.21 (GPIO21)
- new net LCD_DC: U1001.20 (GPIO20)
- new net LCD_MOSI: R1023.2
- new net LCD_RST_N: U1001.25 (GPIO24)
- new net LCD_SCK: R1022.2
- new net LED_PWR_A: D1001.2 (A), R1024.2
- new net LED_STATUS: R1025.1, U1001.58 (GPIO47_ADC7)
- new net LED_ST_A: D1002.2 (A), R1025.2
- new net MCU_LCD_MOSI: R1023.1, U1001.23 (GPIO23)
- new net MCU_LCD_SCK: R1022.1, U1001.22 (GPIO22)
- new net MCU_SWCLK: TP1001.1, U1001.33 (SWCLK)
- new net MCU_SWDIO: TP1002.1, U1001.34 (SWDIO)
- new net MCU_USB_DN: R1008.2
- new net MCU_USB_DP: R1007.2
- new net NTC_ADC0: C1026.1, R1020.2, U1001.53 (GPIO42_ADC2)
- new net NTC_ADC1: C1027.1, R1021.2, U1001.54 (GPIO43_ADC3)
- new net PDIN_INT_N: U1001.4 (GPIO7)
- new net PDIN_PRESENT: U1001.37 (GPIO29)
- new net PMG1_SWCLK: U1001.27 (GPIO26)
- new net PMG1_SWDIO: U1001.28 (GPIO27)
- new net PMG1_XRES_N: U1001.36 (GPIO28)
- new net QSPI_SCLK: U1001.71 (QSPI_SCLK), U1002.6 (CLK)
- new net QSPI_SD0: U1001.72 (QSPI_SD0), U1002.5 (DI)
- new net QSPI_SD1: U1001.74 (QSPI_SD1), U1002.2 (DO)
- new net QSPI_SD2: U1001.73 (QSPI_SD2), U1002.3 (IO2)
- new net QSPI_SD3: U1001.70 (QSPI_SD3), U1002.7 (IO3)
- new net QSPI_SS: R1004.1, R1005.1, U1001.75 (QSPI_SS), U1002.1 (~{CS})
- new net RUN: R1006.1, TP1003.1, U1001.35 (RUN)
- new net RUN_SW: R1006.2, SW1002.1 (A), SW1002.2 (B)
- new net TEMP_ALERT_N: R1016.1, U1003.6 (P2)
- new net UART_RX: J1001.2 (Pin_2), U1001.78 (GPIO1)
- new net UART_TX: J1001.1 (Pin_1), U1001.77 (GPIO0)
- new net USBA1_FORCE_EN: U1001.43 (GPIO34)
- new net USBA1_ISENSE: R1018.1
- new net USBA2_FORCE_EN: U1001.44 (GPIO35)
- new net USBA2_ISENSE: R1019.1
- new net USB_DM_IC: R1008.1, U1001.66 (USB_DM)
- new net USB_DP_IC: R1007.1, U1001.67 (USB_DP)
- new net VREG_AVDD: C1003.1, R1001.2, U1001.61 (VREG_AVDD)
- new net VREG_LX: L1001.1, U1001.63 (VREG_LX)
- new net XIN: C1020.1, U1001.30 (XIN), Y1001.1
- new net XOUT: R1003.1, U1001.31 (XOUT)
- new net XTAL_O: C1021.1, R1003.2, Y1001.3
Other:
- note added: "+1V1 is the RP2350 core (DVDD), made on-chip (VREG_LX -> L1001 -> VREG_FB/DVDD); it is not used elsewhere."
- note added: "1. RP2350B QFN-80 10x10, 0.4 mm pitch, EP = GND (via array). All 48 GPIO allocated (table in docs/design/mcu.md)"
- note added: "10. CROSS-SHEET RULES"
- note added: "2. POWER +3V3 in; internal switching regulator makes +1V1 (DVDD). Copy the RPi minimal-board regulator layout exactly."
- note added: "27R at the RP2350 pins (RPi requirement). Route as a 90R differential pair over solid GND. No VBUS sense: the"
- note added: "3. CLOCK / QSPI FLASH / BOOTSEL / RUN / SWD"
- note added: "4. USB FS -> USB7206C port 6 (USB2-only)"
- note added: "5. I2C PULL-UPS (hub SMBus has none here: HUB_SMB_PU feeds them on usb_hub)"
- note added: "6. I/O EXPANDER TCA9534 @ 0x20 on I2C_SYS: status inputs + PHY reset (48 GPIOs are all used)"
- note added: "7. ADC GPIO40-47 are NOT fault tolerant (max IOVDD + 0.5 V, i.e. 0.5 V with +3V3 off) -> series R on live sources"
- note added: "8. LCD SPI SPI0 (GPIO20-23) at up to 62.5 MHz write clock; series R at the source"
- note added: "9. STATUS LEDs / DEBUG UART"
- note added: "ADC0/1 USBA1/2_ISENSE: INA180A2 (gain 50) output -> 10k + 10 nF. If usb_a powers the INA180 from +5V, its output can"
- note added: "ADC2/3 NTC_ADC0/1: 10k bias from ADC_AVDD, NTC to GND remote. 25 C -> 1/2 ADC_AVDD; 100 C -> ~0.3 V."
- note added: "ADC4/5 HDR_ADC0/1: user header (1k + ESD on display_ui), 0-3.3 V only. ADC_AVDD = 3.3 V reference (internal temp = ch 8)."
- note added: "ADC_AVDD = +3V3 through 10R/4.7u: the ADC reference; NTC bias resistors hang on ADC_AVDD -> ratiometric."
- note added: "All are 0-3.3 V signals that are low or unpowered whenever +3V3 is off -> no level shifting needed. These signals are"
- note added: "BOOTSEL also recovers a hub stuck waiting for SMBus config: hold BOOTSEL + power-cycle -> HUB_SMB_PU stays low."
- note added: "CR_LED from the +5V-powered GL3224) lands on a fault-tolerant GPIO (0-39, <= 3.63 V while unpowered). ADC pins (40-47)"
- note added: "Dead-deck start (PMG1 on laptop VBUS, +3V3 off): every signal that can be high then (PDIN_PRESENT, PMG1_SWDIO/SWCLK pulls,"
- note added: "HUB_SMB_CLK/DAT: no pull-ups here. HUB_SMB_PU: push-pull. HUB_RESET_N, PMG1_XRES_N: drive low or Hi-Z only."
- note added: "I2C_EXT (GPIO30/31) and HUB SMBus (GPIO8/9) run on PIO I2C (clock stretching supported); both pin pairs are also"
- note added: "I2C_SYS = I2C1 (GPIO2/3), I2C_PD = I2C0 (GPIO4/5): hardware controllers, 400 kHz (1 MHz possible on I2C_PD)."
- note added: "J1001 (unpopulated, in_bom no): UART0 115200 8N1 debug console; GPIO0/1 are fault tolerant (FTDI cable safe)."
- note added: "Load: ~30-60 mA at 150 MHz both cores; < 0.2 W."
- note added: "P0 EXT_PWR_PRESENT (3.3 V push-pull, 100k PD on pd_pmg1) P1 LAPTOP_OVP_N (open drain, 10k PU on power_laptop)"
- note added: "P2 TEMP_ALERT_N (TMP1075 wired-OR, 10k PU here) P3/P4 CR_CD_SD_N / CR_CD_USD_N (card detect, pull-ups on card_reader)"
- note added: "P5 ETH_RESET_N (output: write 0 to reset the RTL8156BG; 10k PU here) P6/P7 spare (10k PD; candidates: CCPROT faults)."
- note added: "Place the QSPI_SS resistors next to the flash; keep the QSPI bus short and direct, no stubs."
- note added: "Power LED shows +3V3 even with no/broken firmware; status LED is firmware-driven (blink codes, fault)."
- note added: "RP2350 is always attached to the hub; firmware treats bus reset/suspend as attach/detach."
- note added: "Reset state of all GPIOs = input + ~50k pull-down: FORCE_EN off, LCD in reset, backlight off, SMB_PU low (hub boots stand-alone)."
- note added: "SWD pads (TP1001-TP1004, 1.0 mm, 2.54 mm apart): SWCLK, SWDIO, RUN, GND -> pogo jig or Raspberry Pi Debug Probe."
- note added: "VREG_PGND: own via cluster, return the C6/C7 switching loop straight to pin 62 (RPi datasheet 'External components')."
- note added: "also seen by the PMG1 (EXT_PWR_PRESENT, LAPTOP_OVP_N) which owns the safety reaction; the RP2350 only displays them."
- note added: "exceed 3.3 V or be live before +3V3: 10k limits the clamp current to < 0.2 mA. Prefer INA180 on +3V3 (see mcu.md)."
- note added: "hardware-I2C capable if firmware wants to swap buses. Pull-ups go to +3V3: with +3V3 off (dead-deck start, PMG1 on VBUS)"
- note added: "only see sources that are off with +3V3, or go through >= 1k (ISENSE 10k, header 1k). PMG1_XRES_N has its pass FET on pd_pmg1."
- note added: "the PD bus idles low and no current flows into the unpowered RP2350 (all pins here are fault tolerant up to 3.63 V)."
- note removed: "TODO — planned contents: RP2350B + W25Q128 QSPI, 12MHz xtal, USB2 to hub, I2C buses (PD, sensors, hub SMBus), SWD master to PMG1, BOOTSEL/RESET buttons, 2 user buttons, status LEDs, SWD pads."
- title: odeck-10 — MCU -> odeck-10 — MCU (RP2350B)

Commit message: Schematic review + footprint verification; fix all MAJOR findings
Reviews (docs/review/): power, PD/mux, data path, MCU/UI - 0 blockers,
7 majors, all resolved:
- power: diode-OR inputs (no shutdown-based PD-in priority), sink hand-over
  gated by delayed PG_5V, PD-in capacitance within 100 uF, HV resistor sizes,
  OVP filter/threshold, VBB_PG soft-start qualification
- card reader MS2_INS/SD2_WP phantom card, hub VBUS_DET level buffer
- RP2350 inductor dot text; minors across all sheets (HPD pull-down, PMG1
  INT pin, PHY TX caps, erratum E9 pull-downs, PHY I2C bridge gating,
  backlight 39 ohm, +1V1 cap, IOX P7)
Footprints: all 54 custom footprints checked vs manufacturer drawings,
50 fixed (courtyards, pads, paste, RJ45 mirrored pinout, EP sizes, holes);
removed obsolete FL_001 placeholder.
Firmware rules collected in docs/design/mcu.md.
186 parts, all JLC stock >= 5; netlist verify OK; ERC clean.

Co-Authored-By: Claude Opus 5.5 <noreply@anthropic.com>
Parts:
- added C1028: 4.7u, Capacitor_SMD:C_0402_1005Metric, symbol Device:C
- added R1026, R1027: 1k, Resistor_SMD:R_0402_1005Metric, symbol Device:R
- added R1028: 10k, Resistor_SMD:R_0402_1005Metric, symbol Device:R
Connections:
- net +1V1: now also C1028.1
- net GND: now also C1028.2, R1028.2
- net IOX_P7: now also R1028.1
- net PMG1_SWCLK: now also R1026.2; no longer U1001.27 (GPIO26)
- net PMG1_SWDIO: now also R1027.2; no longer U1001.28 (GPIO27)
- new net MCU_PMG1_SWCLK: R1026.1, U1001.27 (GPIO26)
- new net MCU_PMG1_SWDIO: R1027.1, U1001.28 (GPIO27)
Other:
- note added: "(40-47) only see sources that are off with +3V3, or go through >= 1k (ISENSE 10k, header 10k). PMG1_XRES_N has its pass FET on pd_pmg1."
- note added: "11. FIRMWARE RULES (full list: docs/design/mcu.md 'Firmware rules')"
- note added: "ADC0/1 USBA1/2_ISENSE: INA180A2 (gain 50, on +3V3 with 1k/100 nF on usb_a) -> 10k + 10 nF here: second RC stage,"
- note added: "ADC4/5 HDR_ADC0/1: user header (10k + 10 nF + ESD on display_ui), 0-3.3 V only. ADC_AVDD = 3.3 V reference (internal temp = ch 8)."
- note added: "Dead-deck start (PMG1 on laptop VBUS, +3V3 off): every signal that can be high then (PDIN_PRESENT, PMG1_SWDIO/SWCLK pulls"
- note added: "ETH power cycle via P5 >= 100 ms. HUB_SMB_PU high only with working firmware; AA56h after config."
- note added: "GPIO30/31 to I2C1 = the controllers already used by I2C_PD / I2C_SYS, so a hardware swap costs the other bus."
- note added: "I2C_EXT (GPIO30/31) and HUB SMBus (GPIO8/9) run on PIO I2C (clock stretching supported). GPIO8/9 map to I2C0 and"
- note added: "L1001 ORIENTATION: dot = +1V1/C_OUT side (pad 2), as on the Pico 2 layout (DS Fig. 26); NOT toward VREG_LX. Rotated or"
- note added: "LAPTOP_SNK_EN: reset/flash drops +5V/+3V3, the RP2350 browns out mid-flash and the PMG1 is left bricked."
- note added: "P5 ETH_RESET_N (output: write 0 to reset the RTL8156BG; 10k PU here) P6 ETH_I2C_EN (output; 100k PD R820 on ethernet)"
- note added: "P7 spare (10k PD here; firmware: configure as output low). Candidates: a CCPROT fault or USBA1_OCS_N."
- note added: "PMG1 SWD (GPIO26/27 -> 1k -> PMG1_SWCLK/SWDIO) + PMG1_XRES_N (GPIO28). FIRMWARE RULE: never assert PMG1_XRES_N, start a"
- note added: "PMG1 SWD session or enter the PMG1 I2C bootloader unless EXT_PWR_PRESENT = 1 (TCA9534 P0). Bus-powered, the PMG1 holds"
- note added: "PMG1_XRES_N / PMG1 SWD / PMG1 I2C bootloader: ONLY while EXT_PWR_PRESENT = 1 (bus-powered = PMG1 is the deck's supply)."
- note added: "Pull-ups go to +3V3: with +3V3 off (dead-deck start, PMG1 on VBUS)"
- note added: "Second 4.7u on +1V1 sits at DVDD pin 32 (bottom edge of the package), not next to L1001/C_OUT."
- note added: "TCA9534: configure P7 (spare) as output low; P5/P6 outputs: clear P6 ETH_I2C_EN before driving P5 ETH_RESET_N low."
- note added: "and limits injection into the non-FT pads (< 0.2 mA) should the source ever be live with +3V3 off."
- note added: "pin-swapped = worse regulation. Check the JLC CPL rotation/preview against the footprint dot before ordering."
- note added: "via 1k, CR_LED from the +5V-powered GL3224) lands on a fault-tolerant GPIO (0-39, <= 3.63 V while unpowered). ADC pins"
- note removed: "ADC0/1 USBA1/2_ISENSE: INA180A2 (gain 50) output -> 10k + 10 nF. If usb_a powers the INA180 from +5V, its output can"
- note removed: "ADC4/5 HDR_ADC0/1: user header (1k + ESD on display_ui), 0-3.3 V only. ADC_AVDD = 3.3 V reference (internal temp = ch 8)."
- note removed: "CR_LED from the +5V-powered GL3224) lands on a fault-tolerant GPIO (0-39, <= 3.63 V while unpowered). ADC pins (40-47)"
- note removed: "Dead-deck start (PMG1 on laptop VBUS, +3V3 off): every signal that can be high then (PDIN_PRESENT, PMG1_SWDIO/SWCLK pulls,"
- note removed: "I2C_EXT (GPIO30/31) and HUB SMBus (GPIO8/9) run on PIO I2C (clock stretching supported); both pin pairs are also"
- note removed: "P5 ETH_RESET_N (output: write 0 to reset the RTL8156BG; 10k PU here) P6/P7 spare (10k PD; candidates: CCPROT faults)."
- note removed: "exceed 3.3 V or be live before +3V3: 10k limits the clamp current to < 0.2 mA. Prefer INA180 on +3V3 (see mcu.md)."
- note removed: "hardware-I2C capable if firmware wants to swap buses. Pull-ups go to +3V3: with +3V3 off (dead-deck start, PMG1 on VBUS)"
- note removed: "only see sources that are off with +3V3, or go through >= 1k (ISENSE 10k, header 1k). PMG1_XRES_N has its pass FET on pd_pmg1."
