File: hardware/odeck-10/pd_pmg1.kicad_sch (KiCad schematic)
At the start: 0 parts

Commit message: Draft data-path sheets: PD controller, USB-C muxes/DP, USB hub
- pd_pmg1: PMG1-S3 (CYPM1321, dead-battery Rd) dual-port: laptop EPR source +
  DP UFP_D, downstream 5 V/3 A + DP DFP_D, HPD relay, VBUS-powered cold start,
  I2C 0x42, SWD/reset via cuttable jumpers
- usbc_muxes: laptop + downstream USB-C, TUSB1064/TUSB1046 in GPIO mode,
  TPD4S480 (EPR) / TPD6S300 CC protection, 10G-rated ESD, AC coupling
- usb_hub: USB7206C port map, SMBus-optional boot, reset gated by RAILS_PG,
  BC1.2 on USB-A ports, hub-TX AC caps
- schgen: in_bom option; nets: VBUS_LSW, PMG1_VDDD, hub/mux/CC links
- import_lcsc.sh: guard against overwriting other parts' footprints
- 137 parts, all JLC stock >= 5

Co-Authored-By: Claude Opus 5.5 <noreply@anthropic.com>
Parts:
- added C401, C405, C408, C412, C413: 1u, Capacitor_SMD:C_0402_1005Metric, symbol Device:C
- added C402, C404, C406, C407, C409, C410, C411, C420: 100n, Capacitor_SMD:C_0402_1005Metric, symbol Device:C
- added C403: 4.7u, Capacitor_SMD:C_0603_1608Metric, symbol Device:C
- added C414, C415: 100n/50V, Capacitor_SMD:C_0603_1608Metric, symbol Device:C
- added C416, C417, C418, C419: 390p, Capacitor_SMD:C_0402_1005Metric, symbol Device:C
- added C421, C422: 10u, Capacitor_SMD:C_0805_2012Metric, symbol Device:C
- added JP401, JP402, JP403: SWD_CUT, Jumper:SolderJumper-2_P1.3mm_Bridged_RoundedPad1.0x1.5mm, symbol Jumper:SolderJumper_2_Bridged
- added Q401: AO3400A, Package_TO_SOT_SMD:SOT-23, symbol Transistor_FET:AO3400A
- added Q402: AO4842, Package_SO:SOIC-8_3.9x4.9mm_P1.27mm, symbol Transistor_FET:AO4842
- added R401: 4.7k, Resistor_SMD:R_0402_1005Metric, symbol Device:R
- added R402, R403, R404: 10k, Resistor_SMD:R_0402_1005Metric, symbol Device:R
- added R405, R406, R407, R408, R409, R410, R411, R412: 100k, Resistor_SMD:R_0402_1005Metric, symbol Device:R
- added R413, R414: 1k, Resistor_SMD:R_0402_1005Metric, symbol Device:R
- added R415: 5m, Resistor_SMD:R_1206_3216Metric, symbol Device:R
- added TP401: SWDIO_L, TestPoint:TestPoint_Pad_D1.0mm, symbol Connector:TestPoint
- added TP402: SWCLK_L, TestPoint:TestPoint_Pad_D1.0mm, symbol Connector:TestPoint
- added TP403: XRES, TestPoint:TestPoint_Pad_D1.0mm, symbol Connector:TestPoint
- added TP404: UART_TX, TestPoint:TestPoint_Pad_D1.0mm, symbol Connector:TestPoint
- added TP405: UART_RX, TestPoint:TestPoint_Pad_D1.0mm, symbol Connector:TestPoint
- added TP406: GND, TestPoint:TestPoint_Pad_D1.0mm, symbol Connector:TestPoint
- added U401: CYPM1321-97BZXI, odeck:BGA-97_L6.0-W6.0-P0.50-TL_CYPD8225-97BZXIT, symbol odeck:CYPM1322-97BZXI_C6580811
Connections:
- new net +3V3: C401.1, C402.1, Q401.1 (G), R402.2, R403.2, R404.1, U401.B14 (VSYS)
- new net +5V: C412.1, C413.1, C421.1, R415.1, U401.C15 (CSP_P1), U401.L1 (VCONN_Source_P1), U401.L14 (VCONN_Source_P0), U401.L15 (VCONN_Source_P0), U401.L2 (VCONN_Source_P1)
- new net DS_CC1: C418.1, U401.N1 (CC1_P1), U401.N2 (CC1_P1)
- new net DS_CC2: C419.1, U401.J1 (CC2_P1), U401.J2 (CC2_P1)
- new net DS_FETD: Q402.5 (D2), Q402.6 (D2), Q402.7 (D1), Q402.8 (D1)
- new net DS_GIN: Q402.2 (G1), U401.P2 (VBUS_IN_CTRL_P1)
- new net DS_GOUT: Q402.4 (G2), U401.P1 (VBUS_OUT_CTRL_P1)
- new net DS_HPD: R413.2, U401.M10 (P1.4)
- new net DS_SRC: Q402.1 (S1), R415.2, U401.C14 (CSN_P1), U401.R2 (VBUS_IN_NGDO_P1)
- new net EXT_PWR_PRESENT: R406.1, U401.G15 (P7.0)
- new net GND: C401.2, C402.2, C403.2, C404.2, C405.2, C406.2, C407.2, C408.2, C409.2, C410.2, C411.2, C412.2, C413.2, C414.2, C415.2, C416.2, C417.2, C418.2, C419.2, C420.2, C421.2, C422.2, R405.2, R406.2, R407.2, R408.2, R409.2, R410.2, R411.2, R412.2, TP406.1, U401.F10 (VSS), U401.F12 (VSS), U401.F8 (VSS), U401.H10 (VSS), U401.H8 (VSS), U401.K10 (VSS), U401.K8 (VSS)
- new net HPD0_OUT: R414.1, U401.K4 (P1.3)
- new net HPD1_OUT: R413.1, U401.G14 (P7.1)
- new net I2C_PD_INT_N: R403.1, U401.H4 (P5.5)
- new net I2C_PD_SCL: U401.E15 (P4.0)
- new net I2C_PD_SDA: U401.D12 (P4.1)
- new net LAPTOP_CC1: C416.1, U401.N14 (CC1_P0), U401.N15 (CC1_P0)
- new net LAPTOP_CC2: C417.1, U401.J14 (CC2_P0), U401.J15 (CC2_P0)
- new net LAPTOP_OVP_N: U401.B11 (P7.4)
- new net LAPTOP_SNK_EN: U401.R8 (P0.0)
- new net LAPTOP_SRC_EN: U401.B7 (P2.6)
- new net MUX_DS_CTL0: R410.1, U401.B1 (P3.3)
- new net MUX_DS_CTL1: R411.1, U401.D4 (P3.4)
- new net MUX_DS_FLIP: R412.1, U401.C1 (P3.7)
- new net MUX_UP_CTL0: R407.1, U401.A1 (P3.0)
- new net MUX_UP_CTL1: R408.1, U401.B3 (P3.1)
- new net MUX_UP_FLIP: R409.1, U401.C2 (P3.2)
- new net P3V3_SNS: R404.2, R405.1, U401.A9 (P7.5)
- new net PDIN_PRESENT: U401.A14 (P7.2)
- new net PMG1_SWCLK: JP403.1 (A)
- new net PMG1_SWCLK_L: JP403.2 (B), TP402.1, U401.P3 (P1.1)
- new net PMG1_SWDIO: JP402.1 (A)
- new net PMG1_SWDIO_L: JP402.2 (B), TP401.1, U401.R3 (P1.2)
- new net PMG1_UART_RX: TP405.1, U401.B5 (P2.3)
- new net PMG1_UART_TX: TP404.1, U401.A3 (P2.2)
- new net PMG1_VCCD: C411.1, U401.D10 (VCCD)
- new net PMG1_VDDD: C403.1, C404.1, C405.1, C406.1, C407.1, C408.1, C409.1, C410.1, R401.2, U401.B8 (VDDIO), U401.D6 (VDDA), U401.D8 (VDDD), U401.F6 (VDDA), U401.H12 (VDDIO)
- new net PMG1_XRES: C420.1, Q401.3 (D), R401.1, TP403.1, U401.E14 (XRES)
- new net PMG1_XRES_N: JP401.1 (A)
- new net UP_HPD: R414.2
- new net VBB_EN: U401.A2 (P2.0)
- new net VBB_PG: U401.B13 (P7.3)
- new net VBB_VSEL0: U401.B2 (P2.1)
- new net VBB_VSEL1: U401.A7 (P2.4)
- new net VBB_VSEL2: U401.A5 (P2.5)
- new net VBUS_DS: C415.1, C422.1, Q402.3 (S2), U401.H14 (VBUS_C_P1), U401.R1 (VBUS_OUT_NGDO_P1)
- new net VBUS_LAPTOP: C414.1, U401.A15 (CSN_P0), U401.H15 (VBUS_C_P0)
- new net VBUS_LSW: U401.B15 (CSP_P0)
- new net XRES_RP: JP401.2 (B), Q401.2 (S), R402.1
- no-connect marks 0 -> 33
Other:
- note added: "2. PMG1 SUPPLY (dead-deck capable) VSYS = +3V3 (deck powered): VDDD = VSYS - 0.1 V. Dead deck (no +3V3): the internal 28 V VBUS regulator powers VDDD (3.0-3.65 V, 60 mA max) from VBUS_C_P0 (laptop) or VBUS_C_P1. VSYS has priority. VDDIO and VDDA tied to VDDD (PMG1_VDDD) so EVERY GPIO works in a dead-deck cold start (LAPTOP_SNK_EN is additionally on a VDDD-domain pin, P0.0). Cost: 10 mA total GPIO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"
- note added: "3. CC LINES 390 pF to GND on each CC (Infineon reference; within cReceiver 200-600 pF). CC pins are 6 V abs max: LAPTOP_CC1/2 must arrive through CC OVP (TPD4S480) on usbc_muxes."
- note added: "4. RESET + SWD (RP2350 = SWD programmer; default-closed solder jumpers, cut to isolate) XRES: 4.7k pull-up to VDDD + 100 nF (Infineon Fig. 12). The RP2350 side goes through a pass FET (gate = +3V3, BSS138-style): with +3V3 absent (dead-deck boot) the unpowered RP2350 pin cannot clamp XRES low and hold the PMG1 in reset. With +3V3 present, RP2350 driving PMG1_XRES_N low resets PMG1 (non-inverting;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"
- note added: "5. HOST INTERFACE (RP2350) I2C_PD on SCB0 (P4.0 SCL / P4.1 SDA: the only fail-safe I2C pins, same SCB as the dock example's HPI). PMG1 target address 0x42 (firmware-defined, CCGx HPI alternate address; TPS26750 = 0x21 on the same bus). Bus pull-ups on the MCU sheet (+3V3). I2C_PD_INT_N: P5.5 (datasheet 'embedded controller interrupt'), open-drain, 10k pull-up here. P3V3_SNS (P7.5): +3V3 present (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"
- note added: "6. MUX CONTROL (TUSB1064 / TUSB1046 in GPIO mode, I2C_EN = 0) Port 0 -> TUSB1064: CTL0 = USB3 on, CTL1 = DP on, FLIP = CC orientation (P3.0/P3.1/P3.2). Port 1 -> TUSB1046: CTL0, CTL1, FLIP (P3.3/P3.4/P3.7). 100k pull-downs: PMG1 in reset/unpowered -> muxes default to USB3 off / DP off / no flip. HPD: HPD1_OUT (P7.1, port-1 HPD block, output: follows the monitor's HPD_State/IRQ_HPD Attention) -> 1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"
- note added: "7. PORT 1 (DOWNSTREAM) VBUS SOURCE +5V -> 5 mOhm (CSP_P1/CSN_P1) -> AO4842 back-to-back -> VBUS_DS Gate-driver pair 1 (VBUS_IN_CTRL_P1 = supply-side FET, VBUS_OUT_CTRL_P1 = connector-side FET), common drain: blocks both directions when off (a phone/charger on the port cannot back-feed +5V). Gate overdrive 4.5-10.5 V, OFF VGS down to -VBUS: AO4842 VGS +-20 V, 30 V, 21 mOhm -> 3 A: 0.38 W. CSA 1: O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"
- note added: "PMG1-S3 DUAL-PORT PD CONTROLLER (CYPM1321-97BZXI = CYPM1322 + dead-battery Rd on CC) Port 0 = laptop USB-C: DRP. Source 5-28 V EPR 140 W via power_laptop (VBB_EN, VBB_VSEL2..0, VBB_PG, LAPTOP_SRC_EN); sink in bus-powered mode (LAPTOP_SNK_EN). Data UFP, DP Alt Mode UFP_D -> TUSB1064. The port-0 power path is EXTERNAL (LM74800/LM74502 on power_laptop): PMG1 gate-driver pair 0 is unused, firmware sw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"
- note removed: "TODO — planned contents: Infineon PMG1-S3 CYPM1322-97BZXI: port0 = laptop (EPR source, DP UFP_D, TUSB1064 ctrl), port1 = downstream USB-C (5V/3A source, DP DFP_D, TUSB1046 ctrl, forced-5V mode), HPD relay. SWD to RP2350 through default-closed solder jumper."
- title: odeck-10 — PD controller -> odeck-10 — PD controller PMG1-S3 (laptop + downstream USB-C)

Commit message: Schematic review + footprint verification; fix all MAJOR findings
Reviews (docs/review/): power, PD/mux, data path, MCU/UI - 0 blockers,
7 majors, all resolved:
- power: diode-OR inputs (no shutdown-based PD-in priority), sink hand-over
  gated by delayed PG_5V, PD-in capacitance within 100 uF, HV resistor sizes,
  OVP filter/threshold, VBB_PG soft-start qualification
- card reader MS2_INS/SD2_WP phantom card, hub VBUS_DET level buffer
- RP2350 inductor dot text; minors across all sheets (HPD pull-down, PMG1
  INT pin, PHY TX caps, erratum E9 pull-downs, PHY I2C bridge gating,
  backlight 39 ohm, +1V1 cap, IOX P7)
Footprints: all 54 custom footprints checked vs manufacturer drawings,
50 fixed (courtyards, pads, paste, RJ45 mirrored pinout, EP sizes, holes);
removed obsolete FL_001 placeholder.
Firmware rules collected in docs/design/mcu.md.
186 parts, all JLC stock >= 5; netlist verify OK; ERC clean.

Co-Authored-By: Claude Opus 5.5 <noreply@anthropic.com>
Connections:
- net +3V3: no longer R403.2
- net I2C_PD_INT_N: now also U401.B9 (P7.6); no longer U401.H4 (P5.5)
- net PMG1_VDDD: now also R403.2
Other:
- note added: "5. HOST INTERFACE (RP2350) I2C_PD on SCB0 (P4.0 SCL / P4.1 SDA: the only fail-safe I2C pins, same SCB as the dock example's HPI). PMG1 target address 0x42 (firmware-defined, CCGx HPI alternate address; TPS26750 = 0x21 on the same bus). Bus pull-ups on the MCU sheet (+3V3). I2C_PD_INT_N: P7.6 (B9), open-drain, 10k pull-up to PMG1_VDDD here (never above VDDIO). Not P5.5: ports 2/3/5 carry analog fu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"
- note added: "6. MUX CONTROL (TUSB1064 / TUSB1046 in GPIO mode, I2C_EN = 0) Port 0 -> TUSB1064: CTL0 = USB3 on, CTL1 = DP on, FLIP = CC orientation (P3.0/P3.1/P3.2). Port 1 -> TUSB1046: CTL0, CTL1, FLIP (P3.3/P3.4/P3.7). 100k pull-downs hold CTL0/CTL1/FLIP low while PMG1 is in reset/unpowered. NOTE: both muxes still enter USB3 mode (no flip) at VCC power-up regardless of CTL0 and leave it only on a CTL0 L-H-L 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"
- note removed: "5. HOST INTERFACE (RP2350) I2C_PD on SCB0 (P4.0 SCL / P4.1 SDA: the only fail-safe I2C pins, same SCB as the dock example's HPI). PMG1 target address 0x42 (firmware-defined, CCGx HPI alternate address; TPS26750 = 0x21 on the same bus). Bus pull-ups on the MCU sheet (+3V3). I2C_PD_INT_N: P5.5 (datasheet 'embedded controller interrupt'), open-drain, 10k pull-up here. P3V3_SNS (P7.5): +3V3 present (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"
- note removed: "6. MUX CONTROL (TUSB1064 / TUSB1046 in GPIO mode, I2C_EN = 0) Port 0 -> TUSB1064: CTL0 = USB3 on, CTL1 = DP on, FLIP = CC orientation (P3.0/P3.1/P3.2). Port 1 -> TUSB1046: CTL0, CTL1, FLIP (P3.3/P3.4/P3.7). 100k pull-downs: PMG1 in reset/unpowered -> muxes default to USB3 off / DP off / no flip. HPD: HPD1_OUT (P7.1, port-1 HPD block, output: follows the monitor's HPD_State/IRQ_HPD Attention) -> 1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"
Changed lines of the file:
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@@
 		)
 	)
-	(no_connect
-		(at 473.71 295.91)
+	(wire
+		(pts
+			(xy 473.71 295.91) (xy 476.25 295.91)
+		)
+		(stroke
+			(width 0)
+			(type default)
+		)
+	)
+	(global_label "I2C_PD_INT_N"
+		(shape passive)
+		(at 476.25 295.91 0)
+		(fields_autoplaced yes)
+		(effects
+			(font
+				(size 1.27 1.27)
+			)
+			(justify left)
+		)
+		(property "Intersheetrefs" "${INTERSHEET_REFS}"
+			(at 476.25 295.91 0)
+			(effects
+				(font
+					(size 1.27 1.27)
+				)
+				(hide yes)
+			)
+		)
 	)
 	(wire
@@
 		(at 473.71 191.77)
 	)
-	(wire
-		(pts
-			(xy 473.71 267.97) (xy 476.25 267.97)
-		)
-		(stroke
-			(width 0)
-			(type default)
-		)
-	)
-	(global_label "I2C_PD_INT_N"
-		(shape passive)
-		(at 476.25 267.97 0)
-		(fields_autoplaced yes)
-		(effects
-			(font
-				(size 1.27 1.27)
-			)
-			(justify left)
-		)
-		(property "Intersheetrefs" "${INTERSHEET_REFS}"
-			(at 476.25 267.97 0)
-			(effects
-				(font
-					(size 1.27 1.27)
-				)
-				(hide yes)
-			)
-		)
+	(no_connect
+		(at 473.71 267.97)
 	)
 	(no_connect
@@
 			)
 		)
-		(property "Description" "INT_N pull-up"
+		(property "Description" "INT_N pull-up to VDDIO rail (P7.6)"
 			(at 25.40 345.44 0)
 			(effects
@@
 		)
 	)
-	(global_label "+3V3"
+	(global_label "PMG1_VDDD"
 		(shape passive)
 		(at 25.40 351.79 270)
@@
 		)
 	)
-	(text "5. HOST INTERFACE (RP2350)  I2C_PD on SCB0 (P4.0 SCL / P4.1 SDA: the only fail-safe I2C pins,\n  same SCB as the dock example's HPI). PMG1 target address 0x42 (firmware-defined, CCGx HPI alternate\n  address; TPS26750 = 0x21 on the same bus). Bus pull-ups on the MCU sheet (+3V3).\nI2C_PD_INT_N: P5.5 (datasheet 'embedded controller interrupt'), open-drain, 10k pull-up here.\nP3V3_SNS (P7.5): +3V3 present (10k/100k). Firmware keeps every output towards +3V3-powered chips\n  (mux CTL/FLIP, UP_HPD, DS_HPD, LAPTOP_SRC_EN) low until P3V3_SNS is high (no back-powering).\nEXT_PWR_PRESENT 100k pull-down: its 74LVC1G32 driver is unpowered (Ioff) in a dead deck; without it the\n  net floats - here AND at the power_laptop sink-switch FET gate."
+	(text "5. HOST INTERFACE (RP2350)  I2C_PD on SCB0 (P4.0 SCL / P4.1 SDA: the only fail-safe I2C pins,\n  same SCB as the dock example's HPI). PMG1 target address 0x42 (firmware-defined, CCGx HPI alternate\n  address; TPS26750 = 0x21 on the same bus). Bus pull-ups on the MCU sheet (+3V3).\nI2C_PD_INT_N: P7.6 (B9), open-drain, 10k pull-up to PMG1_VDDD here (never above VDDIO). Not P5.5: ports 2/3/5\n  carry analog functions and must not see an external voltage above VDDIO or before all supplies are up (DS 2.6.3);\n  a +3V3 pull-up sits ~0.1 V above VDDIO (= VDDD = VSYS - 0.1 V). VDDD-referenced high (3.0-3.65 V) is > RP2350 VIH.\n  Dead deck: VDDD up, RP2350 unpowered -> <= 0.35 mA into the RP2350 pad through 10k; PMG1 firmware leaves INT_N\n  released (high) until P3V3_SNS is high, so the RP2350 never sees a spurious edge at boot.\nP3V3_SNS (P7.5): +3V3 present (10k/100k). Firmware keeps every output towards +3V3-powered chips\n  (mux CTL/FLIP, UP_HPD, DS_HPD, LAPTOP_SRC_EN) low until P3V3_SNS is high (no back-powering).\nEXT_PWR_PRESENT 100k pull-down: its 74LVC1G32 driver is unpowered (Ioff) in a dead deck; without it the\n  net floats - here AND at the power_laptop sink-switch FET gate."
 		(exclude_from_sim no)
 		(at 20.32 302.26 0)
@@
 		)
 	)
-	(text "6. MUX CONTROL (TUSB1064 / TUSB1046 in GPIO mode, I2C_EN = 0)\nPort 0 -> TUSB1064: CTL0 = USB3 on, CTL1 = DP on, FLIP = CC orientation (P3.0/P3.1/P3.2).\nPort 1 -> TUSB1046: CTL0, CTL1, FLIP (P3.3/P3.4/P3.7). 100k pull-downs: PMG1 in reset/unpowered ->\n  muxes default to USB3 off / DP off / no flip.\nHPD: HPD1_OUT (P7.1, port-1 HPD block, output: follows the monitor's HPD_State/IRQ_HPD Attention) -> 1k\n  -> DS_HPD -> TUSB1046 HPDIN, and -> P1.4 (port-0 HPD block in receive mode, as a dock's DP sink HPD)\n  -> port 0 sends Attention/Status to the laptop. HPD0_OUT (P1.3, GPIO) -> 1k -> UP_HPD -> TUSB1064\n  HPDIN (DP lanes enabled only while high). 1k: limits injection into the non-fail-safe HPDIN pins."
+	(text "6. MUX CONTROL (TUSB1064 / TUSB1046 in GPIO mode, I2C_EN = 0)\nPort 0 -> TUSB1064: CTL0 = USB3 on, CTL1 = DP on, FLIP = CC orientation (P3.0/P3.1/P3.2).\nPort 1 -> TUSB1046: CTL0, CTL1, FLIP (P3.3/P3.4/P3.7). 100k pull-downs hold CTL0/CTL1/FLIP low while PMG1 is\n  in reset/unpowered. NOTE: both muxes still enter USB3 mode (no flip) at VCC power-up regardless of CTL0 and\n  leave it only on a CTL0 L-H-L pulse (TUSB1064 8.4.1, TUSB1046 7.4.1): firmware pulses CTL0 after P3V3_SNS\n  goes high and on every detach. DP lanes stay off (CTL1 low; TUSB1064 HPDIN 100k PD on usbc_muxes).\nHPD: HPD1_OUT (P7.1, port-1 HPD block, output: follows the monitor's HPD_State/IRQ_HPD Attention) -> 1k\n  -> DS_HPD -> TUSB1046 HPDIN, and -> P1.4 (port-0 HPD block in receive mode, as a dock's DP sink HPD)\n  -> port 0 sends Attention/Status to the laptop. HPD0_OUT (P1.3, GPIO) -> 1k -> UP_HPD -> TUSB1064\n  HPDIN (DP lanes enabled only while high). 1k: limits injection into the non-fail-safe HPDIN pins."
 		(exclude_from_sim no)
 		(at 203.2 12.7 0)
