File: hardware/odeck-10/usb_a.kicad_sch (KiCad schematic)
At the start: 0 parts

Commit message: Draft remaining sheets: USB-A, card reader, Ethernet, MCU, display/UI, sensors
- usb_a: 2x 10G USB-A, TPS2553 switches (hub OR RP2350 force), INA180 sense
- card_reader: GL3224 + SD/microSD, card detect + activity to MCU
- ethernet: RTL8156BG with switched 3.3 V, 0.95 V PWM buck, 2.5G magjack,
  LED buffer, EUI-48 EEPROM + gated I2C bridge for MAC eFuse write
- mcu: RP2350B reference core, full GPIO table, TCA9534 expander, PIO I2C
- display_ui: 2.0" ST7789 LCD + backlight PWM, buttons, unpopulated GPIO
  header (series R + ESD), Qwiic
- sensors: 8x TMP1075, 2 NTCs, thermocouple pads
- integration: ETH_I2C_EN net, TPS62933F for +3V3, PWR_FLAGs
- schgen: deterministic UUIDs; bom_check: cost summary
- 181 parts, all JLC stock >= 5; netlist verify OK; ERC clean but 1 spare pin

Co-Authored-By: Claude Opus 5.5 <noreply@anthropic.com>
Parts:
- added C701, C709: 150u/10V, Capacitor_Tantalum_SMD:CP_EIA-7343-31_Kemet-D, symbol Device:C_Polarized
- added C702, C704, C710, C712: 10u, Capacitor_SMD:C_0805_2012Metric, symbol Device:C
- added C703, C705, C706, C707, C708, C711, C713, C714, C715, C716: 100n, Capacitor_SMD:C_0402_1005Metric, symbol Device:C
- added D701, D703: TPD4E02B04, odeck:USON-10_L2.5-W1.0-P0.50-BL, symbol odeck:TPD4E02B04DQAR
- added D702, D704: USBLC6-2SC6, odeck:SOT-23-6_L2.9-W1.6-P0.95-LS2.8-BL, symbol odeck:USBLC6-2SC6
- added J701, J702: GSB4111312HR, odeck:USB-A-TH_U231-091N-4BLRC19-F1-A, symbol odeck:GSB4111312HR
- added R701, R706: 15k, Resistor_SMD:R_0402_1005Metric, symbol Device:R
- added R702, R703, R707, R708: 100k, Resistor_SMD:R_0402_1005Metric, symbol Device:R
- added R704, R709: 30m, Resistor_SMD:R_0805_2012Metric, symbol Device:R
- added R705, R710: 1k, Resistor_SMD:R_0402_1005Metric, symbol Device:R
- added U701, U704: TPS2553, odeck:SOT-23-6_L2.9-W1.6-P0.95-LS2.8-BR, symbol odeck:TPS2553DBVR
- added U702, U705: SN74LVC1G32, Package_TO_SOT_SMD:SOT-23-5, symbol 74xGxx:74LVC1G32
- added U703, U706: INA180A2, odeck:SOT-23-5_L3.0-W1.7-P0.95-LS2.8-BL, symbol odeck:INA180A2IDBVR
Connections:
- new net +3V3: C706.1, C707.1, C714.1, C715.1, U702.5 (VCC), U703.5 (VS), U705.5 (VCC), U706.5 (VS)
- new net +5V: R704.1, R709.1, U703.3 (IN+), U706.3 (IN+)
- new net +5V_USBA1: C701.1, C702.1, C703.1, D702.5, J701.1 (VBUS), U701.6 (OUT)
- new net +5V_USBA2: C709.1, C710.1, C711.1, D704.5, J702.1 (VBUS), U704.6 (OUT)
- new net GND: C701.2, C702.2, C703.2, C704.2, C705.2, C706.2, C707.2, C708.2, C709.2, C710.2, C711.2, C712.2, C713.2, C714.2, C715.2, C716.2, D701.3 (GND), D701.8 (GND), D702.2, D703.3 (GND), D703.8 (GND), D704.2, J701.10 (EH), J701.11 (EH), J701.4 (GND), J701.7 (GND_DRAIN), J702.10 (EH), J702.11 (EH), J702.4 (GND), J702.7 (GND_DRAIN), R701.2, R702.2, R703.2, R706.2, R707.2, R708.2, U701.2 (GND), U702.3 (GND), U703.2 (GND), U704.2 (GND), U705.3 (GND), U706.2 (GND)
- new net USBA1_DN: D702.3, D702.4, J701.2 (D-)
- new net USBA1_DP: D702.1, D702.6, J701.3 (D+)
- new net USBA1_EN: R703.1, U701.3 (EN), U702.4
- new net USBA1_FORCE_EN: R702.1, U702.2
- new net USBA1_ILIM: R701.1, U701.5 (ILIM)
- new net USBA1_ISENSE: C708.1, R705.2
- new net USBA1_ISNS: R705.1, U703.1 (OUT)
- new net USBA1_OCS_N: U701.4 (/FAULT)
- new net USBA1_PWR_EN: U702.1
- new net USBA1_SS_RXN: D701.5 (IO4), D701.6 (NC), J701.5 (SSRX-)
- new net USBA1_SS_RXP: D701.4 (IO3), D701.7 (NC), J701.6 (SSRX+)
- new net USBA1_SS_TXN: D701.2 (IO2), D701.9 (NC), J701.8 (SSTX-)
- new net USBA1_SS_TXP: D701.1 (IO1), D701.10 (NC), J701.9 (SSTX+)
- new net USBA1_SW_IN: C704.1, C705.1, R704.2, U701.1 (IN), U703.4 (IN-)
- new net USBA2_DN: D704.3, D704.4, J702.2 (D-)
- new net USBA2_DP: D704.1, D704.6, J702.3 (D+)
- new net USBA2_EN: R708.1, U704.3 (EN), U705.4
- new net USBA2_FORCE_EN: R707.1, U705.2
- new net USBA2_ILIM: R706.1, U704.5 (ILIM)
- new net USBA2_ISENSE: C716.1, R710.2
- new net USBA2_ISNS: R710.1, U706.1 (OUT)
- new net USBA2_OCS_N: U704.4 (/FAULT)
- new net USBA2_PWR_EN: U705.1
- new net USBA2_SS_RXN: D703.5 (IO4), D703.6 (NC), J702.5 (SSRX-)
- new net USBA2_SS_RXP: D703.4 (IO3), D703.7 (NC), J702.6 (SSRX+)
- new net USBA2_SS_TXN: D703.2 (IO2), D703.9 (NC), J702.8 (SSTX-)
- new net USBA2_SS_TXP: D703.1 (IO1), D703.10 (NC), J702.9 (SSTX+)
- new net USBA2_SW_IN: C712.1, C713.1, R709.2, U704.1 (IN), U706.4 (IN-)
Other:
- note added: "(port already off at the hub, or hub reports OC). RP2350 sees the fault as ISENSE pinned at ~1.6-1.8 A -> firmware drops FORCE_EN."
- note added: "1. USB-A #1 (hub port 2, PRT_CTL2/PF16)"
- note added: "2. USB-A #2 (hub port 3, PRT_CTL3/PF15)"
- note added: "25 mA auto-off threshold = 37.5 mV out; INA180 offset +-150 uV x50 = +-7.5 mV (~5 mA). Shunt loss 1.8 A: 97 mW."
- note added: "AC coupling (USB 3.2 6.2.x: the cap belongs to the TRANSMITTER's board): hub TX -> 220 nF on usb_hub -> USBAx_SS_TX* -> connector"
- note added: "Connector pin names are the USB-IF host-side names (StdA_SSTX = host transmits): hub TX goes to SSTX, not SSRX."
- note added: "Current limit: RILIM 15.0k -> 1.61 A min / 1.80 A max (TPS2553 DS table): covers BC1.2 DCP/CDP 1.5 A."
- note added: "Current sense: 30 mOhm before the switch (IN side), INA180A2 x50 -> 1.5 V/A; 2.0 A = 3.0 V, full scale 2.2 A at 3.3 V."
- note added: "ESD: TPD4E02B04 (0.25 pF) on the 4 SS lines, USBLC6-2SC6 on D+/D- (clamps to VBUS), all at the connector, flow-through."
- note added: "FAULT# (open drain, 7.5 ms deglitch) -> USBAx_OCS_N = same node as PWR_EN (0R on usb_hub). No pull-up on this node here."
- note added: "Forced port (FORCE_EN high): switch stays on in constant-current limit / thermal cycling; FAULT# only pulls the hub's node"
- note added: "Hub-owned port: FAULT# pulls the node low -> hub reads overcurrent, latches the port off (drives low) -> OR output follows."
- note added: "NOTES"
- note added: "Port power: TPS2553 EN = USBAx_PWR_EN (hub PRT_CTL: ~50k internal pull-up = on, driven low = off) OR USBAx_FORCE_EN (RP2350)."
- note added: "Route IN+/IN- as a Kelvin pair from the inner edges of the shunt pads."
- note added: "SSTX (pins 9/8). Device TX caps are inside the plugged device -> connector SSRX (pins 6/5) -> USBAx_SS_RX* -> hub RX with NO cap here."
- note added: "Shell / EH tabs and GND_DRAIN -> GND directly (no chassis on odeck-10; via-stitch the tabs to all GND planes)."
- note added: "TPS2553 soft start (~1 ms) limits inrush into the bulk; the 10 uF on the switch IN side + +5V rail caps supply the transient."
- note added: "USB-A 10G PORTS 2x Amphenol GSB4111312HR (USB 3.2 Gen2), hub ports 2/3 of the USB7206C (usb_hub sheet)"
- note added: "VBUS bulk 150 uF POSCAP + 10 uF + 100 nF per port at the connector (USB 2.0: >= 120 uF per downstream port)."
- note removed: "TODO — planned contents: 2x Amphenol GSB4111312HR (10G), TPS2553 switches (enable = hub PRTPWR OR RP2350), shunt + INA180A2 current sense -> RP2350 ADC, ESD."
- title: odeck-10 — USB-A ports -> odeck-10 — USB-A 10 Gbps ports (2x), port power, current sense

Commit message: Schematic review + footprint verification; fix all MAJOR findings
Reviews (docs/review/): power, PD/mux, data path, MCU/UI - 0 blockers,
7 majors, all resolved:
- power: diode-OR inputs (no shutdown-based PD-in priority), sink hand-over
  gated by delayed PG_5V, PD-in capacitance within 100 uF, HV resistor sizes,
  OVP filter/threshold, VBB_PG soft-start qualification
- card reader MS2_INS/SD2_WP phantom card, hub VBUS_DET level buffer
- RP2350 inductor dot text; minors across all sheets (HPD pull-down, PMG1
  INT pin, PHY TX caps, erratum E9 pull-downs, PHY I2C bridge gating,
  backlight 39 ohm, +1V1 cap, IOX P7)
Footprints: all 54 custom footprints checked vs manufacturer drawings,
50 fixed (courtyards, pads, paste, RJ45 mirrored pinout, EP sizes, holes);
removed obsolete FL_001 placeholder.
Firmware rules collected in docs/design/mcu.md.
186 parts, all JLC stock >= 5; netlist verify OK; ERC clean.

Co-Authored-By: Claude Opus 5.5 <noreply@anthropic.com>
Parts:
- R702, R707: value 100k -> 4.7k; LCSC C25741 -> C25900
Other:
- note added: "FORCE_EN pull-down 4.7k (not 100k): RP2350 erratum E9 (stepping A2) can leave a pad that was driven high and then"
- note added: "reverted to input latched at ~2.2 V (> LVC1G32 VIH 2.0 V) -> port forced on after a crash/BOOTSEL. Only <= 8.2k defeats"
- note added: "the latch; 4.7k costs 0.7 mA from the push-pull GPIO while forced on (VOH drop negligible at 4 mA drive)."
Changed lines of the file:
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@@
 			)
 		)
-		(property "Value" "100k"
+		(property "Value" "4.7k"
 			(at 147.32 128.27 0)
 			(effects
@@
 			)
 		)
-		(property "Description" "FORCE_EN default off (RP2350 in reset / BOOTSEL)"
+		(property "Description" "FORCE_EN default off (RP2350 in reset / BOOTSEL); 4.7k overrides RP2350-E9 pad latch (~2.2 V)"
 			(at 144.78 127.00 0)
 			(effects
@@
 			)
 		)
-		(property "LCSC" "C25741"
+		(property "LCSC" "C25900"
 			(at 144.78 127.00 0)
 			(effects
@@
 			)
 		)
-		(property "Value" "100k"
+		(property "Value" "4.7k"
 			(at 347.98 128.27 0)
 			(effects
@@
 			)
 		)
-		(property "Description" "FORCE_EN default off (RP2350 in reset / BOOTSEL)"
+		(property "Description" "FORCE_EN default off (RP2350 in reset / BOOTSEL); 4.7k overrides RP2350-E9 pad latch (~2.2 V)"
 			(at 345.44 127.00 0)
 			(effects
@@
 			)
 		)
-		(property "LCSC" "C25741"
+		(property "LCSC" "C25900"
 			(at 345.44 127.00 0)
 			(effects
@@
 		)
 	)
-	(text "Current limit: RILIM 15.0k -> 1.61 A min / 1.80 A max (TPS2553 DS table): covers BC1.2 DCP/CDP 1.5 A."
+	(text "FORCE_EN pull-down 4.7k (not 100k): RP2350 erratum E9 (stepping A2) can leave a pad that was driven high and then"
 		(exclude_from_sim no)
 		(at 20.32 213.36 0)
@@
 		)
 	)
-	(text "Current sense: 30 mOhm before the switch (IN side), INA180A2 x50 -> 1.5 V/A; 2.0 A = 3.0 V, full scale 2.2 A at 3.3 V."
+	(text "  reverted to input latched at ~2.2 V (> LVC1G32 VIH 2.0 V) -> port forced on after a crash/BOOTSEL. Only <= 8.2k defeats"
 		(exclude_from_sim no)
 		(at 20.32 215.9 0)
@@
 		)
 	)
-	(text "  25 mA auto-off threshold = 37.5 mV out; INA180 offset +-150 uV x50 = +-7.5 mV (~5 mA). Shunt loss 1.8 A: 97 mW."
+	(text "  the latch; 4.7k costs 0.7 mA from the push-pull GPIO while forced on (VOH drop negligible at 4 mA drive)."
 		(exclude_from_sim no)
 		(at 20.32 218.44 0)
@@
 		)
 	)
-	(text "  Route IN+/IN- as a Kelvin pair from the inner edges of the shunt pads."
+	(text "Current limit: RILIM 15.0k -> 1.61 A min / 1.80 A max (TPS2553 DS table): covers BC1.2 DCP/CDP 1.5 A."
 		(exclude_from_sim no)
 		(at 20.32 220.98 0)
@@
 		)
 	)
-	(text "VBUS bulk 150 uF POSCAP + 10 uF + 100 nF per port at the connector (USB 2.0: >= 120 uF per downstream port)."
+	(text "Current sense: 30 mOhm before the switch (IN side), INA180A2 x50 -> 1.5 V/A; 2.0 A = 3.0 V, full scale 2.2 A at 3.3 V."
 		(exclude_from_sim no)
 		(at 20.32 223.52 0)
@@
 		)
 	)
-	(text "  TPS2553 soft start (~1 ms) limits inrush into the bulk; the 10 uF on the switch IN side + +5V rail caps supply the transient."
+	(text "  25 mA auto-off threshold = 37.5 mV out; INA180 offset +-150 uV x50 = +-7.5 mV (~5 mA). Shunt loss 1.8 A: 97 mW."
 		(exclude_from_sim no)
 		(at 20.32 226.06 0)
@@
 		)
 	)
-	(text "ESD: TPD4E02B04 (0.25 pF) on the 4 SS lines, USBLC6-2SC6 on D+/D- (clamps to VBUS), all at the connector, flow-through."
+	(text "  Route IN+/IN- as a Kelvin pair from the inner edges of the shunt pads."
 		(exclude_from_sim no)
 		(at 20.32 228.6 0)
@@
 		)
 	)
-	(text "Shell / EH tabs and GND_DRAIN -> GND directly (no chassis on odeck-10; via-stitch the tabs to all GND planes)."
+	(text "VBUS bulk 150 uF POSCAP + 10 uF + 100 nF per port at the connector (USB 2.0: >= 120 uF per downstream port)."
 		(exclude_from_sim no)
 		(at 20.32 231.14 0)
 		(effects
 			(font
+				(size 1.27 1.27)
+			)
+			(justify left top)
+		)
+	)
+	(text "  TPS2553 soft start (~1 ms) limits inrush into the bulk; the 10 uF on the switch IN side + +5V rail caps supply the transient."
+		(exclude_from_sim no)
+		(at 20.32 233.68 0)
+		(effects
+			(font
+				(size 1.27 1.27)
+			)
+			(justify left top)
+		)
+	)
+	(text "ESD: TPD4E02B04 (0.25 pF) on the 4 SS lines, USBLC6-2SC6 on D+/D- (clamps to VBUS), all at the connector, flow-through."
+		(exclude_from_sim no)
+		(at 20.32 236.22 0)
+		(effects
+			(font
+				(size 1.27 1.27)
+			)
+			(justify left top)
+		)
+	)
+	(text "Shell / EH tabs and GND_DRAIN -> GND directly (no chassis on odeck-10; via-stitch the tabs to all GND planes)."
+		(exclude_from_sim no)
+		(at 20.32 238.76 0)
+		(effects
+			(font

Commit message: LCD on 12-pin FPC connector; verify USB-A footprint against Amphenol drawing
- display_ui: Hirose FH34SRJ-12S-0.5SH dual-contact FPC connector (J1103),
  panel pin n -> connector pin 13-n after the 180 deg fold; panel is DNP in BOM
  with a pad-less outline footprint; foam tape 1.5 mm with connector window
- USB-A footprint checked against Amphenol GSB4111xxxHR drawing (added to
  docs/datasheets): shell-leg spacing/offset fixed, board-edge marked;
  renamed to USB-A_Amphenol_GSB4111312HR
- import_lcsc.sh: only upgrade newly imported footprints
- stop tracking __pycache__

Co-Authored-By: Claude Opus 5.5 <noreply@anthropic.com>
Parts:
- J701, J702: footprint odeck:USB-A-TH_U231-091N-4BLRC19-F1-A -> odeck:USB-A_Amphenol_GSB4111312HR
Changed lines of the file:
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@@
 			)
 		)
-		(property "Footprint" "odeck:USB-A-TH_U231-091N-4BLRC19-F1-A"
+		(property "Footprint" "odeck:USB-A_Amphenol_GSB4111312HR"
 			(at 35.56 50.80 0)
 			(effects
@@
 			)
 		)
-		(property "Footprint" "odeck:USB-A-TH_U231-091N-4BLRC19-F1-A"
+		(property "Footprint" "odeck:USB-A_Amphenol_GSB4111312HR"
 			(at 236.22 50.80 0)
 			(effects
