File: hardware/odeck-10/ethernet.kicad_sch (KiCad schematic)
At the start: 0 parts

Commit message: Draft remaining sheets: USB-A, card reader, Ethernet, MCU, display/UI, sensors
- usb_a: 2x 10G USB-A, TPS2553 switches (hub OR RP2350 force), INA180 sense
- card_reader: GL3224 + SD/microSD, card detect + activity to MCU
- ethernet: RTL8156BG with switched 3.3 V, 0.95 V PWM buck, 2.5G magjack,
  LED buffer, EUI-48 EEPROM + gated I2C bridge for MAC eFuse write
- mcu: RP2350B reference core, full GPIO table, TCA9534 expander, PIO I2C
- display_ui: 2.0" ST7789 LCD + backlight PWM, buttons, unpopulated GPIO
  header (series R + ESD), Qwiic
- sensors: 8x TMP1075, 2 NTCs, thermocouple pads
- integration: ETH_I2C_EN net, TPS62933F for +3V3, PWR_FLAGs
- schgen: deterministic UUIDs; bom_check: cost summary
- 181 parts, all JLC stock >= 5; netlist verify OK; ERC clean but 1 spare pin

Co-Authored-By: Claude Opus 5.5 <noreply@anthropic.com>
Parts:
- added C801, C832: 1u, Capacitor_SMD:C_0402_1005Metric, symbol Device:C
- added C802: 1n, Capacitor_SMD:C_0402_1005Metric, symbol Device:C
- added C803, C806, C827, C828: 10u, Capacitor_SMD:C_0603_1608Metric, symbol Device:C
- added C804, C808, C809: 22u, Capacitor_SMD:C_0603_1608Metric, symbol Device:C
- added C805, C807, C810, C812, C813, C814, C817, C818, C819, C823, C824, C825, C829, C831, C838, C839, C840: 100n, Capacitor_SMD:C_0402_1005Metric, symbol Device:C
- added C811, C815, C816, C820, C821, C822, C826, C830: 2.2u, Capacitor_SMD:C_0402_1005Metric, symbol Device:C
- added C833, C834: 20p, Capacitor_SMD:C_0402_1005Metric, symbol Device:C
- added C835, C836: 220n, Capacitor_SMD:C_0402_1005Metric, symbol Device:C
- added C837: 390p, Capacitor_SMD:C_0402_1005Metric, symbol Device:C
- added FB801: 100R@100MHz, Inductor_SMD:L_0805_2012Metric, symbol Device:FerriteBead
- added J801: RJ45 2.5G, odeck:RJ45-TH_DGUK211Q340CD2A4D2, symbol odeck:DGUK211Q340CD2A4D2
- added L801: 1uH, Inductor_SMD:L_Sunlord_SWPA4018S, symbol Device:L
- added Q801: 2N7002DW, Package_TO_SOT_SMD:SOT-363_SC-70-6, symbol Transistor_FET:Q_Dual_NMOS_S1G1D2S2G2D1
- added R801, R803, R820: 100k, Resistor_SMD:R_0402_1005Metric, symbol Device:R
- added R802: 59k, Resistor_SMD:R_0402_1005Metric, symbol Device:R
- added R804: 0, Resistor_SMD:R_0402_1005Metric, symbol Device:R
- added R805: 2.49k, Resistor_SMD:R_0402_1005Metric, symbol Device:R
- added R806, R807, R808, R809, R810, R811, R813, R818, R819: 4.7k, Resistor_SMD:R_0402_1005Metric, symbol Device:R
- added R812, R814, R815: 10k, Resistor_SMD:R_0402_1005Metric, symbol Device:R
- added R816, R817: 510, Resistor_SMD:R_0402_1005Metric, symbol Device:R
- added U801: RTL8156BG-CG, odeck:QFN-56_L6.0-W6.0-P0.35--TL-EP4.7, symbol odeck:RTL8156BG-CG
- added U802: TPS22918, Package_TO_SOT_SMD:SOT-23-6, symbol odeck:TPS22918DBVR
- added U803: TPS62A02A, odeck:SOT-5X3-6_W1.6-L1.2-P0.50-LS1.6-BL, symbol odeck:TPS62A02ADRLR
- added U804: SN74LVC3G17, odeck:VSSOP-8_L2.1-W2.4-P0.50-LS3.2-BR, symbol odeck:SN74LVC3G17DCUR
- added U805: 24AA025E48T-I/OT, Package_TO_SOT_SMD:SOT-23-6, symbol odeck:24AA025E48T-I_OT
- added Y801: 25MHz, Crystal:Crystal_SMD_3225-4Pin_3.2x2.5mm, symbol Device:Crystal_GND24
Connections:
- new net +3V3: C801.1, C839.1, C840.1, U802.1 (VIN), U804.8 (VCC), U805.6 (VCC)
- new net ETH_0V95: C808.1, C809.1, C820.1, C821.1, C822.1, C823.1, C824.1, C825.1, C826.1, C827.1, C828.1, C829.1, C830.1, C831.1, L801.2, R802.1, U801.13 (AVDD09), U801.18 (AVDD09), U801.24 (AVDD09), U801.31 (DVDD09), U801.42 (U3VDD09), U801.52 (U2VDD09), U801.56 (DVDD09), U801.7 (DVDD09)
- new net ETH_0V95_UPS: C832.1, U801.54 (DVDD09_UPS)
- new net ETH_3V3: C803.1, C806.1, C807.1, C810.1, C811.1, C812.1, C813.1, C814.1, C815.1, C816.1, C817.1, C818.1, C819.1, FB801.1, J801.12 (LED_Y+), J801.14 (LED_G+), R806.2, R807.2, R808.2, R809.2, R810.2, R811.2, R812.2, R815.2, R818.2, R819.2, U801.10 (AVDD33_XTAL), U801.17 (AVDD33), U801.21 (AVDD33), U801.25 (AVDD33), U801.36 (DVDD33), U801.51 (U2VDD33), U801.55 (DVDD33_UPS), U802.5 (QOD), U802.6 (VOUT), U803.3 (VIN)
- new net ETH_AVDD33_PLL: C804.1, C805.1, FB801.2, U801.9 (AVDD33)
- new net ETH_CFG_SEQ: R814.1, R815.1, U801.35 (CONFIG_SEQ)
- new net ETH_DN: U801.49 (U2DM)
- new net ETH_DOCK_DET: R808.1, U801.37 (DOCK_DET)
- new net ETH_DP: U801.50 (U2DP)
- new net ETH_EECS: R813.1, U801.30 (EECS/TWSI_SCL)
- new net ETH_FB: R802.2, R803.1, U803.5 (FB)
- new net ETH_GPI: R806.1, U801.2 (GPI)
- new net ETH_GPIO4: R809.1, U801.53 (GPIO4)
- new net ETH_I2C_EN: Q801.2 (G), Q801.5 (G), R820.1
- new net ETH_LANWAKE_N: R807.1, U801.1 (LANWAKEB)
- new net ETH_LED0: U804.7 (1Y)
- new net ETH_LED0_N: R810.1, R816.2, U801.38 (LED0/EEDI/SPISI), U804.1 (1A)
- new net ETH_LED1: U804.5 (2Y)
- new net ETH_LED1_N: R811.1, R817.2, U801.39 (LED1/EESK/SPISCK), U804.3 (2A)
- new net ETH_LED2: U804.2 (3Y)
- new net ETH_LED2_N: R812.1, U801.40 (LED2), U804.6 (3A)
- new net ETH_LEDG_K: J801.13 (LED_G-), R816.1
- new net ETH_LEDY_K: J801.11 (LED_Y-), R817.1
- new net ETH_LSW_CT: C802.1, U802.4 (CT)
- new net ETH_MCT: C837.1, C838.1, J801.5 (CT), J801.6 (CT)
- new net ETH_MDI0_N: J801.2 (TD1-), U801.16 (MDIN0)
- new net ETH_MDI0_P: J801.1 (TD1+), U801.15 (MDIP0)
- new net ETH_MDI1_N: J801.4 (TD2-), U801.20 (MDIN1)
- new net ETH_MDI1_P: J801.3 (TD2+), U801.19 (MDIP1)
- new net ETH_MDI2_N: J801.8 (TD3-), U801.23 (MDIN2)
- new net ETH_MDI2_P: J801.7 (TD3+), U801.22 (MDIP2)
- new net ETH_MDI3_N: J801.10 (TD4-), U801.27 (MDIN3)
- new net ETH_MDI3_P: J801.9 (TD4+), U801.26 (MDIP3)
- new net ETH_RESET_N: U802.3 (ON)
- new net ETH_RSET: R805.1, U801.14 (RSET)
- new net ETH_SCL: Q801.4 (S), R819.1, U801.33 (GPIO2/SCL)
- new net ETH_SDA: Q801.1 (S), R818.1, U801.34 (GPIO1/SDA)
- new net ETH_SS_RXN: C836.2
- new net ETH_SS_RXP: C835.2
- new net ETH_SS_TXN: U801.47 (U3SSRXN)
- new net ETH_SS_TXP: U801.46 (U3SSRXP)
- new net ETH_SW: L801.1, U803.2 (SW)
- new net ETH_SWR_EN: R801.1, U801.5 (POW_EXT_SWR), U803.4 (EN)
- new net ETH_TXN_IC: C836.1, U801.44 (U3SSTXN)
- new net ETH_TXP_IC: C835.1, U801.43 (U3SSTXP)
- new net ETH_XI: C833.1, U801.12 (CKXTAL1), Y801.1
- new net ETH_XO: R804.2, U801.11 (CKXTAL2)
- new net ETH_XO_X: C834.1, R804.1, Y801.3
- new net GND: C801.2, C802.2, C803.2, C804.2, C805.2, C806.2, C807.2, C808.2, C809.2, C810.2, C811.2, C812.2, C813.2, C814.2, C815.2, C816.2, C817.2, C818.2, C819.2, C820.2, C821.2, C822.2, C823.2, C824.2, C825.2, C826.2, C827.2, C828.2, C829.2, C830.2, C831.2, C832.2, C833.2, C834.2, C837.2, C838.2, C839.2, C840.2, J801.15 (SHELL), J801.16 (SHELL), R801.2, R803.2, R805.2, R813.2, R814.2, R820.2, U801.45 (GND), U801.48 (GND), U801.57 (GND), U802.2 (GND), U803.1 (GND), U804.4 (GND), U805.2 (VSS), U805.4 (A1), U805.5 (A0), Y801.2 (G), Y801.4 (G)
- new net I2C_SYS_SCL: Q801.3 (D), U805.1 (SCL)
- new net I2C_SYS_SDA: Q801.6 (D), U805.3 (SDA)
- no-connect marks 0 -> 9
Other:
- note added: "(= eFuse autoload record 'write 6 bytes to OCP 0xC000 / PLA_IDR'). The 7-bit slave address is not in the DS -> bench scan."
- note added: "(LED anode at ETH_3V3, active-low pins, Realtek default); function per LED set by eFuse/driver (OCP 0xDD90)."
- note added: "- Buck (U, L, 2x22u) within 10 mm of the QFN; 0.95 V as a short pour on L1/L3; SW node small, away from MDI and XTAL."
- note added: "- MDI pairs over unbroken GND (L2), stop the planes 1.5 mm before the magjack's cable-side pins (Bob Smith is inside)."
- note added: "- QFN-56 0.35 mm pitch (0.15 mm pads, 0.2 mm gaps): JLC 6-layer OK; EP 4.5 mm in DS, imported footprint has 4.7 mm -> check."
- note added: "- TMP1075 'RJ45/RTL8156' (sensors sheet) between the QFN and the magjack. PHY theta-JA 19 C/W (4L ref board) -> +12 K."
- note added: "1. RTL8156BG-CG USB 3.2 Gen1 (5G) <-> 2.5GBASE-T MAC/PHY, QFN-56 6x6 0.35 mm, EP = GND (via array)"
- note added: "2. POWER ETH_3V3 = +3V3 via TPS22918 (ON = ETH_RESET_N) ETH_0V95 = TPS62A02A (EN = POW_EXT_SWR)"
- note added: "3. DECOUPLING every cap at its pin (0402, short via to the GND EP/plane); bulk per Realtek reference"
- note added: "4. CLOCK / RSET / STRAPS (pull values from Realtek RTL8125B ref + verified open RTL8156B design)"
- note added: "5. USB PHY TX -> 220 nF -> hub RX (hub TX caps on usb_hub)"
- note added: "6. MDI + MAGJACK USAKRO DGUK211Q340CD2A4D2 (2.5G, LEDs)"
- note added: "7. LED BUFFER SN74LVC3G17 -> ETH_LED0..2 (RP2350)"
- note added: "8. MAC ADDRESS 24AA025E48 (EUI-48 at 0xFA-0xFF, I2C_SYS 0x50) + switchable bridge to the PHY I2C slave"
- note added: "9. LAYOUT (board-layout.md: RJ45 back-right corner, RTL8156BG + MAC EEPROM in front of it)"
- note added: "Bridge: with ETH_I2C_EN low the PHY can see I2C_SYS traffic (body diodes) but can never pull I2C_SYS low, and an unpowered PHY"
- note added: "Crystal: same YXC 25 MHz/12 pF part as the hub (shared reel). Keep XI/XO short, GND guard, no traces under it."
- note added: "DVDD09_UPS (54) is an INTERNAL LDO output: 1 uF only, never tie to the 0.95 V rail."
- note added: "ETH_LEDx = PHY LEDx level, i.e. ACTIVE LOW (low = LED lit) with the default LED polarity. The jack LEDs load LED0/1,"
- note added: "ETH_RESET_N (TCA9534 P5 on mcu, 10k PU there): high/hi-Z = PHY powered -> Ethernet works with a dead/blank RP2350."
- note added: "Firmware: hold low >= 100 ms (t4 >= 50 ms + QOD discharge). Also usable to turn 2.5GbE off for thermal derating."
- note added: "Hub port 4 (ETH_*): longest SS run on the board (around the hub's PF side). 90 Ohm diff, caps near the PHY,"
- note added: "Jack: 1CT:1CT 2.5G magnetics, 4x75R + 1nF/2kV Bob Smith inside, green LED left / yellow right (pins 14/13, 12/11)."
- note added: "LVC inputs are 5.5 V tolerant with no clamp to VCC, so they never back-power ETH_3V3."
- note added: "Loss: 0.95 V x 0.65 A / ~85 % -> ~0.11 W in the buck; PHY total ~0.6-0.65 W typ (sensors sheet: TMP1075 'RJ45/RTL8156')."
- note added: "MDIx -> TDx+1: MDI0=BI_DA (RJ 1/2), MDI1=BI_DB (3/6), MDI2=BI_DC (4/5), MDI3=BI_DD (7/8). 100 Ohm diff pairs, length-"
- note added: "NC: 3/4/6 (BGS-only regulator pins), CKOUT, LED3, GPIO3, EEDO/SPISO, TWSI_SDA/SPICSB (no EEPROM/flash on the PHY)."
- note added: "No extra ESD on MDI: the magnetics give 2250 VDC isolation and the Realtek reference has none."
- note added: "PHY unpowered (ETH_RESET_N low): inputs sit at 0 V (pull-ups on the dead ETH_3V3) -> outputs low; firmware ignores them."
- note added: "Pin 9 (AVDD33 next to the XTAL) is fed through a ferrite bead (PLL supply, Realtek ref 'AVDD33_PLL')."
- note added: "Plan: RP2350 reads the EUI-48 from U805 (0x50, 0xFA..0xFF), powers the PHY, sets ETH_I2C_EN, writes the OTP code ONCE (eFuse is"
- note added: "RTL8156BG 0.95 V: 0.92-0.98 V (+-3 %), 364 mA typ / 650 mA max; rise 0.5-2.2 ms; off->on >= 50 ms (DS table 25/27)."
- note added: "RTL8156BG MAC sources (DS 6.4/6.6): internal eFuse/OTP (>= 512 B autoload) or an external 93C46/TWSI EEPROM, the latter"
- note added: "Shell -> GND (odeck convention: no separate chassis; via-stitch both shell pins). LEDs are low-side driven by the PHY"
- note added: "Straps/pulls go to ETH_3V3 (never +3V3) so nothing back-powers the PHY while ETH_RESET_N holds it off."
- note added: "TPS62A02A = forced-PWM variant (Realtek: switcher feeding the PHY must run PWM >= 1 MHz); 1 ms soft start meets t3."
- note added: "The buck runs from ETH_3V3, so ETH_RESET_N low also kills 0.95 V; EN = POW_EXT_SWR (PHY output, 100k PD)."
- note added: "VOUT = 0.6 V x (1 + 59k/100k) = 0.954 V; VFB +-1.5 % + 1 % resistors -> 0.932-0.977 V worst case (inside window)."
- note added: "crossings use the PHY's MDI-swap option (eFuse/register) instead of vias."
- note added: "is not back-fed. Enable only while ETH_3V3 is on (else the dead 4.7k pull-ups would hold I2C_SYS low)."
- note added: "matched within pair, no vias if possible, no planes under the magjack's cable side. If the QFN-to-jack order forces"
- note added: "modified via the I2C function' = I2C SLAVE on GPIO1/SDA + GPIO2/SCL, 36-byte 'OTP code': [addr] 25 C0 00 MAC0..MAC5 + 26x 00"
- note added: "one-time; each rewrite burns ~36 B of the 512 B), clears ETH_I2C_EN and logs it. Fallbacks: host tool (Realtek PG tool /"
- note added: "only after a Realtek PG-tool eFuse command selects it; blank eFuse -> chip defaults (no unique MAC). DS 6.6: 'MACID can be"
- note added: "rtunicpg) programs the same EUI-48 over USB (RP2350 reports it in the status app), or the OS overrides the MAC at runtime."
- note added: "so the RP2350 must not read those pins directly; the buffers also isolate the MCU from the switched PHY rail."
- note added: "symmetric, L2 void under the 0402 pads. USB2 ETH_DP/DN: 90 Ohm, no series parts. The PHY is Gen1 (5 Gbps)."
- note removed: "TODO — planned contents: RTL8156BG-CG 2.5GbE, USAKRO DGUK211Q340CD2A4D2 RJ45, LED pins -> RP2350, 24AA02E48 EUI-48 MAC EEPROM."
- title: odeck-10 — Ethernet -> odeck-10 — 2.5 GbE (RTL8156BG)

Commit message: Schematic review + footprint verification; fix all MAJOR findings
Reviews (docs/review/): power, PD/mux, data path, MCU/UI - 0 blockers,
7 majors, all resolved:
- power: diode-OR inputs (no shutdown-based PD-in priority), sink hand-over
  gated by delayed PG_5V, PD-in capacitance within 100 uF, HV resistor sizes,
  OVP filter/threshold, VBB_PG soft-start qualification
- card reader MS2_INS/SD2_WP phantom card, hub VBUS_DET level buffer
- RP2350 inductor dot text; minors across all sheets (HPD pull-down, PMG1
  INT pin, PHY TX caps, erratum E9 pull-downs, PHY I2C bridge gating,
  backlight 39 ohm, +1V1 cap, IOX P7)
Footprints: all 54 custom footprints checked vs manufacturer drawings,
50 fixed (courtyards, pads, paste, RJ45 mirrored pinout, EP sizes, holes);
removed obsolete FL_001 placeholder.
Firmware rules collected in docs/design/mcu.md.
186 parts, all JLC stock >= 5; netlist verify OK; ERC clean.

Co-Authored-By: Claude Opus 5.5 <noreply@anthropic.com>
Parts:
- added C841: 100n, Capacitor_SMD:C_0402_1005Metric, symbol Device:C
- added R821: 100k, Resistor_SMD:R_0402_1005Metric, symbol Device:R
- added U806: 74LVC1G17, Package_TO_SOT_SMD:SOT-23-5, symbol 74xGxx:74LVC1G17
- C835, C836: value 220n -> 100n; LCSC C16772 -> C1525
- Q801: value 2N7002DW -> BSS138DW; LCSC C83571 -> C154900; MPN (none) -> BSS138DW-7-F
Connections:
- net ETH_3V3: now also C841.1, U806.5 (VCC)
- net ETH_I2C_EN: now also U806.2; no longer Q801.2 (G), Q801.5 (G)
- net GND: now also C841.2, R821.2, U806.3 (GND)
- new net ETH_BR_G: Q801.2 (G), Q801.5 (G), R821.1, U806.4
- no-connect marks 9 -> 10
Other:
- note added: "0x48-0x4F/0x50); confirm the OTP write persists (write once, power-cycle via ETH_RESET_N, read PLA_IDR over USB) and that"
- note added: "5. USB PHY TX -> 100 nF -> hub RX (hub TX caps on usb_hub)"
- note added: "Bench items (review data #5): scan I2C_SYS with the bridge on vs off (PHY address, collisions with 0x20/0x41/0x44/0x45/"
- note added: "Bridge: with the gates low the PHY can see I2C_SYS traffic (body diodes) but can never pull I2C_SYS low, and an unpowered PHY"
- note added: "Gen1 C_AC_COUPLING = 75-200 nF -> 100 nF (same as the GL3224 TX); 220 nF is only valid for Gen2 transmitters."
- note added: "I2C_SYS into the dead PHY pull-ups and lock the TCA9534 that controls both (review mcu_ui #5). Firmware should still"
- note added: "be high while ETH_3V3 is up (driver unpowered -> Ioff, 100k holds the gates low; VOH <= ETH_3V3 while it decays, QOD"
- note added: "clear P6 before powering the PHY down. Q801 = BSS138DW (VGS(th) <= 1.5 V) for solid conduction with a 3.3 V gate."
- note added: "is not back-fed. Gate drive ETH_BR_G = 74LVC1G17 powered from ETH_3V3, input ETH_I2C_EN (TCA9534 P6): the gates can only"
- note added: "symmetric, L2 void under the 0402 pads. USB2 ETH_DP/DN: 90 Ohm, no series parts. The PHY is Gen1 (5 Gbps):"
- note added: "takes it to 0 V). So ETH_I2C_EN = 1 with ETH_RESET_N = 0 (firmware bug, thermal power-down mid-write) can no longer drag"
- note added: "the slave answers on a blank eFuse. Volatile write -> rely on the host-tool / OS fallbacks."
- note removed: "5. USB PHY TX -> 220 nF -> hub RX (hub TX caps on usb_hub)"
- note removed: "Bridge: with ETH_I2C_EN low the PHY can see I2C_SYS traffic (body diodes) but can never pull I2C_SYS low, and an unpowered PHY"
- note removed: "is not back-fed. Enable only while ETH_3V3 is on (else the dead 4.7k pull-ups would hold I2C_SYS low)."
- note removed: "symmetric, L2 void under the 0402 pads. USB2 ETH_DP/DN: 90 Ohm, no series parts. The PHY is Gen1 (5 Gbps)."

Commit message: Cost pass, PCB sync + rough placement, renders, README
- cost pass: extended parts 129 -> 114 (~$45/order less), nets unchanged
- tools/pcbsync.py: scripted update-PCB-from-schematic (keeps placed parts)
- tools/set_outline.py; board grown to 130x85 mm (provisional)
- hardware/odeck-10/placement.py: edge connectors + anchor-based packing,
  small passives spill to bottom; all 796 parts on the board (2 at anchor)
- docs/images: top/bottom/iso renders of the rough placement
- README.md: overview, architecture, repo layout, workflow, roadmap

Co-Authored-By: Claude Opus 5.5 <noreply@anthropic.com>
Parts:
- C837: LCSC C76967 -> C282239
Changed lines of the file:
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@@
 			)
 		)
-		(property "LCSC" "C76967"
+		(property "LCSC" "C282239"
 			(at 457.20 88.90 0)
 			(effects
