File: hardware/odeck-10/power_input.kicad_sch (KiCad schematic)
At the start: 0 parts

Commit message: Draft power sheets (input, laptop output, rails) and BOM stock audit
- power_input: TPS26750/TPD4S480 EPR sink, LM74800 PD-in and barrel paths
  (reverse/OV/UV), hardware PD-in priority, EXT_PWR_PRESENT, INA237 VIN monitor
- power_laptop: LM51770 buck-boost 5-28 V x 5 A with VSEL-only voltage steps,
  gated source switch, interlocked bus-power sink, latched 30.8 V OVP, INA226
- power_rails: LM5148 5 V/8 A with ideal-diode backfeed blocking, TPS62933
  3.3 V and 1.15 V, INA226
- tools/bom_check.py: JLC-stock-only audit (>=5); all 116 parts pass
- schgen fixes: multi-line notes, PWR_FLAG skipped in verify, import --force
- docs: design notes per sheet, I2C map, cross-sheet integration items

Co-Authored-By: Claude Opus 5.5 <noreply@anthropic.com>
Parts:
- added C101, C124, C125, C126, C127: 2.2u/100V, Capacitor_SMD:C_1210_3225Metric, symbol Device:C
- added C102, C103, C112, C115, C116: 100n/100V, Capacitor_SMD:C_0603_1608Metric, symbol Device:C
- added C104: 1u, Capacitor_SMD:C_0402_1005Metric, symbol Device:C
- added C105, C113, C117: 100n/50V, Capacitor_SMD:C_0603_1608Metric, symbol Device:C
- added C106, C107, C108: 10u, Capacitor_SMD:C_0603_1608Metric, symbol Device:C
- added C109, C110: 220p, Capacitor_SMD:C_0603_1608Metric, symbol Device:C
- added C111, C119, C120, C121, C128: 100n, Capacitor_SMD:C_0402_1005Metric, symbol Device:C
- added C114, C118: 47n/100V, Capacitor_SMD:C_0603_1608Metric, symbol Device:C
- added C122, C123: 100u/80V, odeck:CAP-SMD_BD10.0-L10.3-W10.3-LS10.8-FD, symbol odeck:RVT100UF80V167RV0112
- added D101: SMCJ51A, odeck:SMC_L6.9-W5.9-LS7.9-RD, symbol odeck:SMCJ51A_C408371
- added D102: SMCJ48CA, odeck:SMC_L6.9-W5.9-LS7.9-BI, symbol odeck:SMCJ48CA_C408370
- added D103: 1N4148W, Diode_SMD:D_SOD-123, symbol Device:D
- added J101: USB-C PD-in, odeck:USB-C-TH_DX07S024XJ1R1100-1, symbol odeck:DX07S024XJ1R1100
- added J102: PJ-063BH, odeck:DC-IN_PJ-063BH, symbol odeck:PJ-063BH_C3095900
- added Q101, Q102, Q103, Q108: 2N7002, Package_TO_SOT_SMD:SOT-23, symbol Transistor_FET:2N7002
- added Q104, Q105, Q106, Q107: BSC026N08NS5, odeck:PG-TDSON-8_L5.0-W6.0-P1.27-BL-EP, symbol odeck:BSC026N08NS5ATMA1
- added R101, R106, R107: 10k, Resistor_SMD:R_0402_1005Metric, symbol Device:R
- added R102, R103, R104, R105, R110, R111, R112, R113, R114, R115, R116, R118, R119, R120, R121, R125, R127, R132, R136: 100k, Resistor_SMD:R_0402_1005Metric, symbol Device:R
- added R108, R109, R122: 2.2k, Resistor_SMD:R_0402_1005Metric, symbol Device:R
- added R117: 1k, Resistor_SMD:R_0402_1005Metric, symbol Device:R
- added R123, R124: 100, Resistor_SMD:R_0402_1005Metric, symbol Device:R
- added R126: 4.7k, Resistor_SMD:R_0402_1005Metric, symbol Device:R
- added R128: 22k, Resistor_SMD:R_0402_1005Metric, symbol Device:R
- added R129, R133: 1M, Resistor_SMD:R_0402_1005Metric, symbol Device:R
- added R130: 33k, Resistor_SMD:R_0402_1005Metric, symbol Device:R
- added R131: 15k, Resistor_SMD:R_0402_1005Metric, symbol Device:R
- added R134: 47k, Resistor_SMD:R_0402_1005Metric, symbol Device:R
- added R135: 7.5k, Resistor_SMD:R_0402_1005Metric, symbol Device:R
- added R137: 2m, Resistor_SMD:R_2512_6332Metric, symbol Device:R
- added TP101: I2Cc_SDA, TestPoint:TestPoint_Pad_D1.0mm, symbol Connector:TestPoint
- added TP102: I2Cc_SCL, TestPoint:TestPoint_Pad_D1.0mm, symbol Connector:TestPoint
- added U101: TPD4S480, odeck:WQFN-20_L3.0-W3.0-P0.40-BL-EP1.7, symbol odeck:TPD4S480RUKR_C43131250
- added U102: TPS26750, odeck:QFN-32_L4.0-W4.0-P0.40-BL-EP2.8, symbol odeck:TPS26750SRSMR_C42166327
- added U103: AT24C512C, odeck:SOIC-8_L4.9-W3.9-P1.27-LS6.0-BL, symbol odeck:AT24C512C-SSHD-T
- added U104, U105: LM74800-Q1, odeck:WSON-12_L3.0-W3.0-P0.50-TL-EP-2, symbol odeck:LM74800QDRRRQ1
- added U106, U107: TLV6700, odeck:TSOT-23-6_L2.9-W1.6-P0.95-LS2.8-BR, symbol odeck:TLV6700DDCR
- added U108: SN74LVC1G32, Package_TO_SOT_SMD:SOT-23-5, symbol 74xGxx:74LVC1G32
- added U109: INA237, odeck:VSSOP-10_L3.0-W3.0-P0.50-LS4.9-BL, symbol odeck:INA237AIDGSR
Connections:
- new net +3V3: C106.1, C119.1, C120.1, C121.1, C128.1, R106.2, R132.2, R136.2, U102.32 (VIN_3V3), U106.5 (VDD), U107.5 (VDD), U108.5 (VCC), U109.1 (A1), U109.2 (A0), U109.6 (VS)
- new net BAR_CAP: C117.1, U105.11 (CAP)
- new net BAR_DGATE: Q106.4 (G), U105.1 (DGATE)
- new net BAR_DVDT: C118.1, R124.2
- new net BAR_EN: Q108.3 (D), R127.2, R128.1, U105.6 (EN/UVLO)
- new net BAR_HGATE: Q107.4 (G), R124.1, U105.8 (HGATE)
- new net BAR_MID: C116.1, C117.2, Q106.5 (D), Q106.6 (D), Q106.7 (D), Q106.8 (D), Q107.5 (D), Q107.6 (D), Q107.7 (D), Q107.8 (D), U105.10 (VS), U105.12 (C)
- new net BAR_MON_OV: R130.2, R131.1, U106.4 (INB-)
- new net BAR_MON_TOP: D103.1 (K), R129.1
- new net BAR_MON_UV: R129.2, R130.1, U106.3 (INA+)
- new net BAR_OK: R132.1, U106.1 (OUTA), U106.6 (OUTB), U108.1
- new net BAR_OV: R125.2, R126.1, U105.5 (OV)
- new net BAR_SW: R125.1, U105.4 (SW)
- new net EXT_PWR_PRESENT: U108.4
- new net GND: C101.2, C102.2, C103.2, C104.2, C105.2, C106.2, C107.2, C108.2, C109.2, C110.2, C111.2, C112.2, C114.2, C115.2, C116.2, C118.2, C119.2, C120.2, C121.2, C122.2, C123.2, C124.2, C125.2, C126.2, C127.2, C128.2, D101.2 (A), D102.2, J101.0, J101.A1 (GND), J101.A12 (GND), J101.B1 (GND), J101.B12 (GND), J102.2, Q101.2 (S), Q102.2 (S), Q103.2 (S), Q108.2 (S), R103.2, R105.2, R110.2, R111.2, R112.2, R113.2, R114.2, R115.2, R116.2, R118.2, R122.2, R126.2, R128.2, R131.2, R135.2, U101.13 (GND), U101.18 (GND), U101.21 (EP), U101.8 (GND), U102.11 (GND), U102.12 (GND), U102.14 (GND), U102.19 (GND), U102.28 (PP5V), U102.29 (PP5V), U102.33 (GND), U103.1 (A0), U103.2 (A1), U103.3 (A2), U103.4 (GND), U103.7 (WP), U104.7 (GND), U105.7 (GND), U106.2 (GND), U107.2 (GND), U108.3 (GND), U109.7 (GND)
- new net I2C_PD_SCL: U102.9 (I2Ct_SCL)
- new net I2C_PD_SDA: U102.8 (I2Ct_SDA)
- new net I2C_SYS_SCL: U109.5 (SCL)
- new net I2C_SYS_SDA: U109.4 (SDA)
- new net PDIN_CC1: C109.1, U101.12 (CC1), U102.24 (CC1)
- new net PDIN_CC2: C110.1, U101.11 (CC2), U102.25 (CC2)
- new net PDIN_C_CC1: J101.A5 (CC1), U101.4 (C_CC1), U101.7 (RPD_G1)
- new net PDIN_C_CC2: J101.B5 (CC2), U101.5 (C_CC2), U101.6 (RPD_G2)
- new net PDIN_EPR_EN: R118.1, U101.16 (EPR_EN), U102.5 (GPIO0)
- new net PDIN_FLT_N: R101.1, U101.9 (~{FLT}), U102.7 (GPIO2)
- new net PDIN_INT_N: R106.1, U102.10 (~{I2Ct_IRQ})
- new net PDIN_PRESENT: R117.2
- new net PDIN_PRES_L: Q108.1 (G), R116.1, R117.1, U102.6 (GPIO1)
- new net PDIN_VBIAS: C103.1, U101.3 (VBIAS)
- new net PDIN_VBUS_LV: C105.1, U101.19 (VBUS_LV), U102.26 (VBUS), U102.27 (VBUS)
- new net PD_ADCIN1: R102.2, R103.1, U102.2 (ADCIN1)
- new net PD_ADCIN2: R104.2, R105.1, U102.3 (ADCIN2)
- new net PD_CAP: C113.1, U104.11 (CAP)
- new net PD_DGATE: Q104.4 (G), U104.1 (DGATE)
- new net PD_DVDT: C114.1, R123.2
- new net PD_GPIO11: R115.1, U102.13 (GPIO11)
- new net PD_GPIO3: R110.1, U102.18 (GPIO3)
- new net PD_GPIO4: R111.1, U102.22 (GPIO4/USB_P/LD1)
- new net PD_GPIO5: R112.1, U102.23 (GPIO5/USB_N/LD2)
- new net PD_GPIO6: R113.1, U102.31 (GPIO6)
- new net PD_GPIO7: R114.1, U102.30 (GPIO7)
- new net PD_HGATE: Q105.4 (G), R123.1, U104.8 (HGATE)
- new net PD_I2CC_IRQ_N: R107.1, U102.17 (~{I2Cc_IRQ})
- new net PD_I2CC_SCL: R109.1, TP102.1, U102.16 (I2Cc_SCL), U103.6 (SCL)
- new net PD_I2CC_SDA: R108.1, TP101.1, U102.15 (I2Cc_SDA), U103.5 (SDA)
- new net PD_LDO_1V5: C108.1, U102.4 (LDO_1V5)
- new net PD_LDO_3V3: C104.1, C107.1, C111.1, R101.2, R102.1, R104.1, R107.2, R108.2, R109.2, R119.2, R120.2, U101.10 (VPWR), U102.1 (LDO_3V3), U103.8 (VCC)
- new net PD_MID: C112.1, C113.2, Q104.5 (D), Q104.6 (D), Q104.7 (D), Q104.8 (D), Q105.5 (D), Q105.6 (D), Q105.7 (D), Q105.8 (D), U104.10 (VS), U104.12 (C)
- new net PD_MON_OV: R134.2, R135.1, U107.4 (INB-)
- new net PD_MON_UV: R133.2, R134.1, U107.3 (INA+)
- new net PD_OK: Q103.3 (D), R136.1, U107.1 (OUTA), U107.6 (OUTB), U108.2
- new net PD_OV: R121.2, R122.1, U104.5 (OV)
- new net PD_OV_TOP: R121.1, U104.4 (SW)
- new net PD_PP_EN_HV: Q101.1 (G), U102.20 (POWER_PATH_EN)
- new net PD_PP_EN_INV: Q101.3 (D), Q102.1 (G), Q103.1 (G), R119.1
- new net PD_SINK_EN: Q102.3 (D), R120.1, U104.6 (EN/UVLO)
- new net VBAR: C115.1, D102.1, D103.2 (A), J102.1, Q106.1 (S), Q106.2 (S), Q106.3 (S), R127.1, U105.2 (A), U105.3 (VSNS)
- new net VBUS_PDIN: C101.1, C102.1, D101.1 (C), J101.A4 (VBUS), J101.A9 (VBUS), J101.B4 (VBUS), J101.B9 (VBUS), Q104.1 (S), Q104.2 (S), Q104.3 (S), R133.1, U101.20 (VBUS), U104.2 (A), U104.3 (VSNS)
- new net VIN: C122.1, C123.1, C124.1, C125.1, C126.1, C127.1, R137.2, U109.8 (VBUS), U109.9 (IN–)
- new net VIN_OR: Q105.1 (S), Q105.2 (S), Q105.3 (S), Q107.1 (S), Q107.2 (S), Q107.3 (S), R137.1, U104.9 (OUT), U105.9 (OUT), U109.10 (IN+)
- no-connect marks 0 -> 24
Other:
- note added: "(SafeMode alternative: ADCIN1 -> LDO_3V3, ADCIN2 -> GND = 7/0, address 0x20.)"
- note added: "-> deck boots from a 5 V-only PD-in even with a blank EEPROM; RP2350 can then program it."
- note added: "1. PD-IN USB-C (power only)"
- note added: "2. TPS26750 EPR SINK CONTROLLER (TI SLVSH67 Fig. 8-24 reference)"
- note added: "3. PD-IN SINK PATH VBUS_PDIN -> VIN_OR"
- note added: "4. BARREL INPUT 9-24 V / 8 A (Same Sky PJ-063BH, 5.5x2.5 mm, pin 1 = centre +)"
- note added: "5. EXT_PWR_PRESENT = BAR_OK OR PD_OK (from the input side, never from VIN)"
- note added: "6. VIN (9-50 V) VIN_OR -> 2 mOhm shunt -> VIN"
- note added: "A 5 V-only PD contract therefore does NOT count as external power."
- note added: "ADCIN1 = ADCIN2 = 100k/100k (decoded 5/5): 'AlwaysEnableSink', I2C target index #2 = 0x21."
- note added: "All of it runs from +3V3, which exists whenever anything powers the deck."
- note added: "BAR_OK: TLV6700 window on VBAR (via 1N4148W, blocks reverse polarity), 1M/33k/15k ladder:"
- note added: "Bulk: 2x 100 uF / 80 V electrolytic + 4x 2.2 uF / 100 V X7R 1210 (VIN reaches 50.4 V)."
- note added: "CURRENT_LSB = 20.48 A / 2^15 = 625 uA. Bidirectional: shows backfeed too. Kelvin-route IN+/IN-."
- note added: "Conduction: 5 A x 2 x 2.6 mOhm = 0.13 W."
- note added: "Config/patch from AT24C512C (64 KB >= 36 KB req.) at 0x50 on the private I2Cc bus."
- note added: "Downstream converters add their own input ceramics on their sheets."
- note added: "EN/UVLO = PD_SINK_EN: path closes only when the TPS26750 enables its sink path."
- note added: "EPR_BLK_G unused (no 5 V source FET: sink-only port). SBU channels unused."
- note added: "GPIO0 = EPR_EN (to TPD4S480), GPIO1 = PDIN_PRESENT (config: high while sink contract active),"
- note added: "GPIO2 = TPD4S480 FLT# input, other GPIOs strapped to GND through 100k (datasheet: tie low if unused)."
- note added: "I2C_PD pull-ups live on the MCU sheet; PDIN_INT_N pull-up here."
- note added: "INA237 (85 V CM, 16-bit, pin-compatible with INA228/INA238) on I2C_SYS at 0x45 (A1 = A0 = VS)."
- note added: "INA237AIDGSR C2864837 (JLC stock 5k). ALERT unused."
- note added: "Inrush: HGATE 55 uA into 47 nF -> 1.17 V/ms. Conduction: 8.3 A x 2 x 2.6 mOhm = 0.36 W."
- note added: "Inrush: HGATE 55 uA into 47 nF -> 1.17 V/ms; ~0.6 A into 500 uF of VIN capacitance."
- note added: "JAE DX07S024XJ1R1100 (48 V / 5 A EPR-rated, C134113). Only VBUS, CC, GND, shell used:"
- note added: "LM74800-Q1 (same as PD path) instead of LM74720: the LM74720 PD pin pulls the HSFET gate to GND,"
- note added: "LM74800-Q1 ideal diode (Q104, DGATE) + load switch (Q105, HGATE), common drain, 2x BSC026N08NS5 80 V."
- note added: "MS mounting tabs left unconnected (would short to + on a reversed plug if tied to GND)."
- note added: "OV: 100k/2.2k -> 1.231 V x 102.2/2.2 = 57.2 V (55.5-58.9 V) > 50.4 V EPR max."
- note added: "OV: 100k/4.7k -> 1.231 V x 104.7/4.7 = 27.4 V (26.6-28.2 V), recovers at 25.2 V."
- note added: "Open-drain outputs wired-AND per source, pull-ups to +3V3; 74LVC1G32 OR -> EXT_PWR_PRESENT."
- note added: "PD_OK: TLV6700 window on VBUS_PDIN, 1M/47k/7.5k: UV 7.7 V, OV 56.2 V, AND sink path on (Q103)."
- note added: "POWER_PATH_EN BUFFER (Fig. 8-5)"
- note added: "PP5V tied to GND: sink-only port, no 5 V sourcing / VCONN (verify with TI)."
- note added: "Powered from +3V3 (VIN_3V3) when the deck runs, else from VBUS via its internal LDO (dead battery)."
- note added: "Q101: inverts POWER_PATH_EN, Q102: PD_SINK_EN (LM74800 EN),"
- note added: "Q103: pulls PD_OK low while the sink path is off."
- note added: "Q106 = ideal diode (DGATE, blocks reverse polarity to -65 V), Q107 = OV / UVLO / enable cut-off (HGATE)."
- note added: "Q108 pulls EN/UVLO low when PDIN_PRESENT (PD-in priority, hardware only)."
- note added: "RP2350 updates it through the TPS26750 host interface (I2Ct, 0x21); I2Cc test pads for recovery."
- note added: "Reverse/backfeed from VIN (barrel or buck-boost) blocked by Q104 (ideal diode)."
- note added: "SMCJ48CA bidirectional TVS: survives a reversed 24 V and a wrong 48 V brick (VBR 53.3 V min)."
- note added: "Shell tied to GND. SMCJ51A TVS: VRWM 51 V > 50.4 V EPR max, VBR 56.7-62.7 V."
- note added: "Shunt 2 mOhm 2512 1 %: 8.3 A -> 16.6 mV, 0.14 W; ADCRANGE=1 (+-40.96 mV) -> +-20.5 A FS,"
- note added: "TPD4S480: CC short-to-VBUS (63 V) protection, dead-battery Rd (RPD_Gx tied to C_CCx),"
- note added: "USB2 D+/D-, SBU and SS pins are left open (no data on this port; no BC1.2)."
- note added: "UV = 0.4 x 1048/48 + 0.5 = 9.2 V, OV = 0.4 x 1048/15 + 0.5 = 28.4 V (~barrel OV 27.4 V)."
- note added: "UVLO: 100k/22k -> 1.231 V x 122/22 = 6.8 V rising, 6.3 V falling."
- note added: "VBUS -> VBUS_LV scaler (x0.42 in EPR) so the TPS26750 VBUS pin (22 V max) can sense 48 V."
- note added: "i.e. Vgs = -VIN while PD-in holds VIN up; the LM74800 HGATE is referenced to OUT."
- note removed: "TODO — planned contents: Inputs & OR-ing: PD-in USB-C (JAE DX07S024XJ1R1100) + TPS26750/TPD4S480 EPR sink, barrel PJ-063BH + LM74720 (reverse/OVP), LM74700/LM74800 on PD-in, PD-in>barrel priority, laptop-VBUS sink switch for bus-powered mode -> 5V rail."
- title: odeck-10 — Power input -> odeck-10 — Power input (PD-in, barrel, VIN)

Commit message: Schematic review + footprint verification; fix all MAJOR findings
Reviews (docs/review/): power, PD/mux, data path, MCU/UI - 0 blockers,
7 majors, all resolved:
- power: diode-OR inputs (no shutdown-based PD-in priority), sink hand-over
  gated by delayed PG_5V, PD-in capacitance within 100 uF, HV resistor sizes,
  OVP filter/threshold, VBB_PG soft-start qualification
- card reader MS2_INS/SD2_WP phantom card, hub VBUS_DET level buffer
- RP2350 inductor dot text; minors across all sheets (HPD pull-down, PMG1
  INT pin, PHY TX caps, erratum E9 pull-downs, PHY I2C bridge gating,
  backlight 39 ohm, +1V1 cap, IOX P7)
Footprints: all 54 custom footprints checked vs manufacturer drawings,
50 fixed (courtyards, pads, paste, RJ45 mirrored pinout, EP sizes, holes);
removed obsolete FL_001 placeholder.
Firmware rules collected in docs/design/mcu.md.
186 parts, all JLC stock >= 5; netlist verify OK; ERC clean.

Co-Authored-By: Claude Opus 5.5 <noreply@anthropic.com>
Parts:
- removed C126, C127: 2.2u/100V, Capacitor_SMD:C_1210_3225Metric, symbol Device:C
- removed C128: 100n, Capacitor_SMD:C_0402_1005Metric, symbol Device:C
- removed Q108: 2N7002, Package_TO_SOT_SMD:SOT-23, symbol Transistor_FET:2N7002
- C122: value 100u/80V -> 47u/100V; footprint odeck:CAP-SMD_BD10.0-L10.3-W10.3-LS10.8-FD -> Capacitor_SMD:CP_Elec_10x10; symbol odeck:RVT100UF80V167RV0112 -> Device:C_Polarized; LCSC C5246576 -> C371305; MPN RVT100UF80V167RV0112 -> (none)
- C123: value 100u/80V -> 1u/100V; footprint odeck:CAP-SMD_BD10.0-L10.3-W10.3-LS10.8-FD -> Capacitor_SMD:C_0805_2012Metric; symbol odeck:RVT100UF80V167RV0112 -> Device:C; LCSC C5246576 -> C126585; MPN RVT100UF80V167RV0112 -> (none)
- C124: value 2.2u/100V -> 100n/100V; footprint Capacitor_SMD:C_1210_3225Metric -> Capacitor_SMD:C_0603_1608Metric; LCSC C153036 -> C15725
- C125: value 2.2u/100V -> 100n; footprint Capacitor_SMD:C_1210_3225Metric -> Capacitor_SMD:C_0402_1005Metric; LCSC C153036 -> C1525
- D101: value SMCJ51A -> 5.0SMDJ51A; LCSC C408371 -> C2990373; MPN SMCJ51A -> 5.0SMDJ51A
- D102: value SMCJ48CA -> 5.0SMDJ48CA; LCSC C408370 -> C2649886; MPN SMCJ48CA -> 5.0SMDJ48CA
- R108, R109: value 2.2k -> 4.7k; LCSC C25879 -> C25900
- R117: value 1k -> 47k; LCSC C11702 -> C25792
- R121, R125, R127: footprint Resistor_SMD:R_0402_1005Metric -> Resistor_SMD:R_0805_2012Metric; LCSC C25741 -> C149504
- R129, R133: footprint Resistor_SMD:R_0402_1005Metric -> Resistor_SMD:R_0805_2012Metric; LCSC C26083 -> C17514
- R130: value 33k -> 39k; LCSC C25779 -> C25783
Connections:
- net +3V3: now also C125.1
- net VIN: no longer C125.1
Other:
- note added: "5.0SMDJ48CA bidirectional TVS (5 kW): survives a reversed 24 V and a wrong 48 V brick (VBR 53.3 V min)."
- note added: "Always armed (no priority): PD-in and barrel are both ideal-diode ORed, the higher voltage feeds VIN."
- note added: "BAR_OK: TLV6700 window on VBAR (via 1N4148W, blocks reverse polarity), 1M/39k/15k ladder (0805 top):"
- note added: "Blank EEPROM: sink path closes at 5 V but PD stays off until a host loads a config, and 5 V on VIN"
- note added: "GPIO0 = EPR_EN (to TPD4S480), GPIO1 = PDIN_PRESENT (informational only, 47k series: <= 60 uA into an"
- note added: "Inrush: HGATE 55 uA into 47 nF -> 1.17 V/ms; ~0.12 A into <= 100 uF of VIN capacitance."
- note added: "Meaning: VIN is (or is about to be) supplied >= ~8 V by PD-in or barrel. Both paths are always armed, so"
- note added: "NO hardware PD-in priority: barrel and PD-in are both always-armed ideal diodes, the higher voltage"
- note added: "Rdyn ~0.32 Ohm -> ~64 V at 5 A, ~68 V at 18 A (SMCJ51A: 82 V). Residual risk vs TPD4S480 63 V: see doc."
- note added: "Shell tied to GND. 5.0SMDJ51A TVS (5 kW, SMC): VRWM 51 V > 50.4 V EPR max, VBR 56.7-62.7 V,"
- note added: "The 47 uF R-C branch damps cable L vs the converter ceramics: peak Zout <= 0.5 Ohm << Zin,min 1.35 Ohm."
- note added: "The laptop sink switch is released only when EXT_PWR_PRESENT AND PG_5V (power_laptop), so a"
- note added: "UV = 0.4 x 1054/54 + 0.4 = 8.2 V (8.0-8.5 V: a 9 V -5 % brick counts), OV = 0.4 x 1054/15 + 0.4 = 28.5 V."
- note added: "VIN capacitance budget (USB PD cSnkBulkPd <= 100 uF, everything the PD source charges when the sink path"
- note added: "VIN capacitance seen by the PD source <= 100 uF (cSnkBulkPd) incl. downstream converter inputs: see doc."
- note added: "does NOT start the LM5148 (UVLO 8 V). First EEPROM programming needs barrel, laptop bus power or I2Cc pads."
- note added: "either OK term implies that input actually feeds VIN (no priority shutdown can make it lie)."
- note added: "is on): here 47 uF/100 V alu (damping, ESR ~0.1-0.6 Ohm) + 1 uF/100 V + 100 nF; power_laptop and"
- note added: "power_rails 4x 4.7 uF/100 V each (no electrolytics there). Total ~90 uF at 20 V, <= 99 uF at 5 V worst."
- note added: "slightly early EXT_PWR_PRESENT (VIN still ramping) never browns out the deck."
- note added: "supplies VIN, so a hand-over never collapses VIN. Source preference = firmware policy (request a PD"
- note added: "unpowered PMG1/RP2350 pin; config: high while sink contract active),"
- note added: "voltage above the barrel to prefer PD-in). Divider tops on VBAR/SW are 0805 (150 V)."
- note removed: "-> deck boots from a 5 V-only PD-in even with a blank EEPROM; RP2350 can then program it."
- note removed: "BAR_OK: TLV6700 window on VBAR (via 1N4148W, blocks reverse polarity), 1M/33k/15k ladder:"
- note removed: "Bulk: 2x 100 uF / 80 V electrolytic + 4x 2.2 uF / 100 V X7R 1210 (VIN reaches 50.4 V)."
- note removed: "Downstream converters add their own input ceramics on their sheets."
- note removed: "GPIO0 = EPR_EN (to TPD4S480), GPIO1 = PDIN_PRESENT (config: high while sink contract active),"
- note removed: "Inrush: HGATE 55 uA into 47 nF -> 1.17 V/ms; ~0.6 A into 500 uF of VIN capacitance."
- note removed: "Q108 pulls EN/UVLO low when PDIN_PRESENT (PD-in priority, hardware only)."
- note removed: "SMCJ48CA bidirectional TVS: survives a reversed 24 V and a wrong 48 V brick (VBR 53.3 V min)."
- note removed: "Shell tied to GND. SMCJ51A TVS: VRWM 51 V > 50.4 V EPR max, VBR 56.7-62.7 V."
- note removed: "UV = 0.4 x 1048/48 + 0.5 = 9.2 V, OV = 0.4 x 1048/15 + 0.5 = 28.4 V (~barrel OV 27.4 V)."
- moved on the sheet: C124, C125

Commit message: Cost pass, PCB sync + rough placement, renders, README
- cost pass: extended parts 129 -> 114 (~$45/order less), nets unchanged
- tools/pcbsync.py: scripted update-PCB-from-schematic (keeps placed parts)
- tools/set_outline.py; board grown to 130x85 mm (provisional)
- hardware/odeck-10/placement.py: edge connectors + anchor-based packing,
  small passives spill to bottom; all 796 parts on the board (2 at anchor)
- docs/images: top/bottom/iso renders of the rough placement
- README.md: overview, architecture, repo layout, workflow, roadmap

Co-Authored-By: Claude Opus 5.5 <noreply@anthropic.com>
Parts:
- C102, C103, C112, C115, C116, C124: footprint Capacitor_SMD:C_0603_1608Metric -> Capacitor_SMD:C_0805_2012Metric; LCSC C15725 -> C28233
- R130: footprint Resistor_SMD:R_0402_1005Metric -> Resistor_SMD:R_0603_1608Metric; LCSC C25783 -> C23153
- R135: footprint Resistor_SMD:R_0402_1005Metric -> Resistor_SMD:R_0603_1608Metric; LCSC C25918 -> C23234
- R137: LCSC C844691 -> C459679; MPN WSL25122L000FEA18 -> RLP25FEGR002
Changed lines of the file:
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@@
 			)
 		)
-		(property "Footprint" "Capacitor_SMD:C_0603_1608Metric"
+		(property "Footprint" "Capacitor_SMD:C_0805_2012Metric"
 			(at 93.98 81.28 0)
 			(effects
@@
 			)
 		)
-		(property "LCSC" "C15725"
+		(property "LCSC" "C28233"
 			(at 93.98 81.28 0)
 			(effects
@@
 			)
 		)
-		(property "Footprint" "Capacitor_SMD:C_0603_1608Metric"
+		(property "Footprint" "Capacitor_SMD:C_0805_2012Metric"
 			(at 124.46 116.84 0)
 			(effects
@@
 			)
 		)
-		(property "LCSC" "C15725"
+		(property "LCSC" "C28233"
 			(at 124.46 116.84 0)
 			(effects
@@
 			)
 		)
-		(property "Footprint" "Capacitor_SMD:C_0603_1608Metric"
+		(property "Footprint" "Capacitor_SMD:C_0805_2012Metric"
 			(at 419.10 132.08 0)
 			(effects
@@
 			)
 		)
-		(property "LCSC" "C15725"
+		(property "LCSC" "C28233"
 			(at 419.10 132.08 0)
 			(effects
@@
 			)
 		)
-		(property "Footprint" "Capacitor_SMD:C_0603_1608Metric"
+		(property "Footprint" "Capacitor_SMD:C_0805_2012Metric"
 			(at 78.74 261.62 0)
 			(effects
@@
 			)
 		)
-		(property "LCSC" "C15725"
+		(property "LCSC" "C28233"
 			(at 78.74 261.62 0)
 			(effects
@@
 			)
 		)
-		(property "Footprint" "Capacitor_SMD:C_0603_1608Metric"
+		(property "Footprint" "Capacitor_SMD:C_0805_2012Metric"
 			(at 195.58 271.78 0)
 			(effects
@@
 			)
 		)
-		(property "LCSC" "C15725"
+		(property "LCSC" "C28233"
 			(at 195.58 271.78 0)
 			(effects
@@
 			)
 		)
-		(property "Footprint" "Resistor_SMD:R_0402_1005Metric"
+		(property "Footprint" "Resistor_SMD:R_0603_1608Metric"
 			(at 314.96 276.86 0)
 			(effects
@@
 			)
 		)
-		(property "LCSC" "C25783"
+		(property "LCSC" "C23153"
 			(at 314.96 276.86 0)
 			(effects
@@
 			)
 		)
-		(property "Footprint" "Resistor_SMD:R_0402_1005Metric"
+		(property "Footprint" "Resistor_SMD:R_0603_1608Metric"
 			(at 403.86 276.86 0)
 			(effects
@@
 			)
 		)
-		(property "LCSC" "C25918"
+		(property "LCSC" "C23234"
 			(at 403.86 276.86 0)
 			(effects
@@
 			)
 		)
-		(property "Footprint" "Capacitor_SMD:C_0603_1608Metric"
+		(property "Footprint" "Capacitor_SMD:C_0805_2012Metric"
 			(at 91.44 393.70 0)
 			(effects
@@
 			)
 		)
-		(property "LCSC" "C15725"
+		(property "LCSC" "C28233"
 			(at 91.44 393.70 0)
 			(effects
@@
 			)
 		)
-		(property "LCSC" "C844691"
+		(property "LCSC" "C459679"
 			(at 132.08 393.70 0)
 			(effects
@@
 			)
 		)
-		(property "MPN" "WSL25122L000FEA18"
+		(property "MPN" "RLP25FEGR002"
 			(at 132.08 393.70 0)
 			(effects
