File: hardware/odeck-10/usb_hub.kicad_sch (KiCad schematic)
At the start: 0 parts

Commit message: Draft data-path sheets: PD controller, USB-C muxes/DP, USB hub
- pd_pmg1: PMG1-S3 (CYPM1321, dead-battery Rd) dual-port: laptop EPR source +
  DP UFP_D, downstream 5 V/3 A + DP DFP_D, HPD relay, VBUS-powered cold start,
  I2C 0x42, SWD/reset via cuttable jumpers
- usbc_muxes: laptop + downstream USB-C, TUSB1064/TUSB1046 in GPIO mode,
  TPD4S480 (EPR) / TPD6S300 CC protection, 10G-rated ESD, AC coupling
- usb_hub: USB7206C port map, SMBus-optional boot, reset gated by RAILS_PG,
  BC1.2 on USB-A ports, hub-TX AC caps
- schgen: in_bom option; nets: VBUS_LSW, PMG1_VDDD, hub/mux/CC links
- import_lcsc.sh: guard against overwriting other parts' footprints
- 137 parts, all JLC stock >= 5

Co-Authored-By: Claude Opus 5.5 <noreply@anthropic.com>
Parts:
- added C601, C602, C603, C604, C605, C606, C607, C608, C609, C610, C611, C612: 220n, Capacitor_SMD:C_0402_1005Metric, symbol Device:C
- added C613, C614, C615, C616, C617, C618, C619, C620, C624, C625, C626, C627, C628, C629, C630, C631, C632, C640: 100n, Capacitor_SMD:C_0402_1005Metric, symbol Device:C
- added C621, C622, C633, C634, C635: 4.7u, Capacitor_SMD:C_0402_1005Metric, symbol Device:C
- added C623, C636, C639: 1n, Capacitor_SMD:C_0402_1005Metric, symbol Device:C
- added C637, C638: 20p, Capacitor_SMD:C_0402_1005Metric, symbol Device:C
- added D601, D602: BAT54WS, Diode_SMD:D_SOD-323, symbol Device:D_Schottky
- added R601: 12k, Resistor_SMD:R_0402_1005Metric, symbol Device:R
- added R602, R603, R604, R605, R609, R614, R624, R627, R628: 10k, Resistor_SMD:R_0402_1005Metric, symbol Device:R
- added R606, R607, R608: 200k, Resistor_SMD:R_0402_1005Metric, symbol Device:R
- added R610, R611, R612, R613, R615, R616, R617, R618, R619, R620, R621, R622, R623, R629: 100k, Resistor_SMD:R_0402_1005Metric, symbol Device:R
- added R625, R626: 47k, Resistor_SMD:R_0402_1005Metric, symbol Device:R
- added R630, R631: 0, Resistor_SMD:R_0402_1005Metric, symbol Device:R
- added U601: USB7206CT/KDX, odeck:VQFN-100_L12.0-W12.0-P0.40-TL-EP8.0, symbol odeck:USB7206CT_KDX
- added U602: SST26VF016B, odeck:SOP-8_L4.9-W3.9-P1.27-LS6.0-BL, symbol odeck:SST26VF016B-104I_SN
- added Y601: 25MHz, Crystal:Crystal_SMD_3225-4Pin_3.2x2.5mm, symbol Device:Crystal_GND24
Connections:
- new net +1V15: C624.1, C625.1, C626.1, C627.1, C628.1, C629.1, C630.1, C631.1, C632.1, C633.1, C634.1, C635.1, C636.1, U601.18 (VCORE), U601.25 (VCORE), U601.31 (VCORE), U601.38 (VCORE), U601.55 (VCORE), U601.78 (VCORE), U601.85 (VCORE), U601.9 (VCORE), U601.93 (VCORE)
- new net +3V3: C613.1, C614.1, C615.1, C616.1, C617.1, C618.1, C619.1, C620.1, C621.1, C622.1, C623.1, C640.1, D602.1 (K), R602.2, R603.2, R604.2, R608.2, R609.2, R614.2, R624.2, U601.26 (VDD33), U601.43 (VDD33), U601.53 (VDD33), U601.62 (VDD33), U601.67 (VDD33), U601.79 (VDD33), U601.88 (VDD33), U601.99 (VDD33), U602.8 (VDD)
- new net CR_DN: U601.6 (USB2DN_DM1/~{PRT_DIS_M1})
- new net CR_DP: U601.5 (USB2DN_DP1/~{PRT_DIS_P1})
- new net CR_SS_RXN: U601.11 (USB3DN_RXDM1)
- new net CR_SS_RXP: U601.10 (USB3DN_RXDP1)
- new net CR_SS_TXN: C604.2
- new net CR_SS_TXP: C603.2
- new net ETH_DN: U601.35 (USB2DN_DM4/~{PRT_DIS_M4})
- new net ETH_DP: U601.34 (USB2DN_DP4/~{PRT_DIS_P4})
- new net ETH_SS_RXN: U601.40 (USB3DN_RXDM4)
- new net ETH_SS_RXP: U601.39 (USB3DN_RXDP4)
- new net ETH_SS_TXN: C610.2
- new net ETH_SS_TXP: C609.2
- new net GND: C613.2, C614.2, C615.2, C616.2, C617.2, C618.2, C619.2, C620.2, C621.2, C622.2, C623.2, C624.2, C625.2, C626.2, C627.2, C628.2, C629.2, C630.2, C631.2, C632.2, C633.2, C634.2, C635.2, C636.2, C637.2, C638.2, C639.2, C640.2, R601.2, R605.2, R606.2, R607.2, R610.2, R611.2, R612.2, R613.2, R615.2, R616.2, R617.2, R618.2, R619.2, R620.2, R621.2, R622.2, R623.2, R626.2, R629.2, U601.101 (VSS), U601.24 (TESTEN), U602.4 (VSS), Y601.2 (G), Y601.4 (G)
- new net HUB_CFG1: R605.1, U601.21 (~{CFG_STRAP1})
- new net HUB_CFG2: R606.1, U601.22 (~{CFG_STRAP2})
- new net HUB_CFG3: R607.1, U601.23 (~{CFG_STRAP3})
- new net HUB_DSC_DN: U601.82 (USB2DN_DM5/~{PRT_DIS_M5})
- new net HUB_DSC_DP: U601.81 (USB2DN_DP5/~{PRT_DIS_P5})
- new net HUB_DSC_SS_RXN: U601.87 (USB3DN_RXDM5)
- new net HUB_DSC_SS_RXP: U601.86 (USB3DN_RXDP5)
- new net HUB_DSC_SS_TXN: C612.2
- new net HUB_DSC_SS_TXP: C611.2
- new net HUB_P1_TXN_IC: C604.1, U601.8 (USB3DN_TXDM1)
- new net HUB_P1_TXP_IC: C603.1, U601.7 (USB3DN_TXDP1)
- new net HUB_P2_TXN_IC: C606.1, U601.17 (USB3DN_TXDM2)
- new net HUB_P2_TXP_IC: C605.1, U601.16 (USB3DN_TXDP2)
- new net HUB_P3_TXN_IC: C608.1, U601.30 (USB3DN_TXDM3)
- new net HUB_P3_TXP_IC: C607.1, U601.29 (USB3DN_TXDP3)
- new net HUB_P4_TXN_IC: C610.1, U601.37 (USB3DN_TXDM4)
- new net HUB_P4_TXP_IC: C609.1, U601.36 (USB3DN_TXDP4)
- new net HUB_P5_TXN_IC: C612.1, U601.84 (USB3DN_TXDM5)
- new net HUB_P5_TXP_IC: C611.1, U601.83 (USB3DN_TXDP5)
- new net HUB_PF18: R620.1, U601.61 (PF18)
- new net HUB_PF19: R621.1, U601.66 (PF19)
- new net HUB_PF29: R623.1, U601.74 (PF29)
- new net HUB_PF3: R615.1, U601.44 (PF3)
- new net HUB_PF31: R622.1, U601.3 (PF31)
- new net HUB_PF4: R616.1, U601.45 (PF4)
- new net HUB_PF5: R617.1, U601.46 (PF5)
- new net HUB_PF6: R618.1, U601.47 (PF6)
- new net HUB_PF7: R619.1, U601.48 (PF7)
- new net HUB_RBIAS: R601.1, U601.100 (RBIAS)
- new net HUB_RESET_N: C639.1, D601.2 (A), R624.1, U601.1 (RESET_N)
- new net HUB_SMB_CLK: R627.1, U601.75 (PF26)
- new net HUB_SMB_DAT: R628.1, U601.76 (PF27)
- new net HUB_SMB_PU: R627.2, R628.2, R629.1
- new net HUB_SPI_CE_N: R608.1, U601.69 (SPI_CE_N/~{CFG_NON_REM}/PF20), U602.1 (~{CE})
- new net HUB_SPI_CLK: R610.1, U601.68 (SPI_CLK/PF21), U602.6 (SCK)
- new net HUB_SPI_D0: R609.1, U601.70 (SPI_D0/~{CFG_BC_EN}/PF22), U602.5 (SI/SIO0)
- new net HUB_SPI_D1: R611.1, U601.71 (SPI_D1/PF23), U602.2 (SO/SIO1)
- new net HUB_SPI_D2: R612.1, U601.72 (SPI_D2/PF24), U602.3 (~{WP}/SIO2)
- new net HUB_SPI_D3: R613.1, R614.1, U601.73 (SPI_D3/PF25), U602.7 (HOLD/SIO3)
- new net HUB_TEST1: R602.1, U601.63 (TEST1)
- new net HUB_TEST2: R603.1, U601.64 (TEST2)
- new net HUB_TEST3: R604.1, U601.65 (TEST3)
- new net HUB_UP_SS_RXN: U601.95 (USB3UP_RXDM)
- new net HUB_UP_SS_RXP: U601.94 (USB3UP_RXDP)
- new net HUB_UP_SS_TXN: C602.2
- new net HUB_UP_SS_TXP: C601.2
- new net HUB_UP_TXN_IC: C602.1, U601.92 (USB3UP_TXDM)
- new net HUB_UP_TXP_IC: C601.1, U601.91 (USB3UP_TXDP)
- new net HUB_VBUS_DET: D602.2 (A), R625.2, R626.1, U601.2 (PF30/VBUS_MON_UP)
- new net HUB_XI: C637.1, U601.98 (XTALI/CLK_IN), Y601.1
- new net HUB_XO: C638.1, U601.97 (XTALO), Y601.3
- new net LAPTOP_USB_DN: U601.90 (USB2UP_DM)
- new net LAPTOP_USB_DP: U601.89 (USB2UP_DP)
- new net MCU_USB_DN: U601.41 (USB2DN_DM6/~{PRT_DIS_M6})
- new net MCU_USB_DP: U601.42 (USB2DN_DP6/~{PRT_DIS_P6})
- new net RAILS_PG: D601.1 (K)
- new net USBA1_DN: U601.15 (USB2DN_DM2/~{PRT_DIS_M2})
- new net USBA1_DP: U601.14 (USB2DN_DP2/~{PRT_DIS_P2})
- new net USBA1_OCS_N: R630.2
- new net USBA1_PWR_EN: R630.1, U601.59 (PF16)
- new net USBA1_SS_RXN: U601.20 (USB3DN_RXDM2)
- new net USBA1_SS_RXP: U601.19 (USB3DN_RXDP2)
- new net USBA1_SS_TXN: C606.2
- new net USBA1_SS_TXP: C605.2
- new net USBA2_DN: U601.28 (USB2DN_DM3/~{PRT_DIS_M3})
- new net USBA2_DP: U601.27 (USB2DN_DP3/~{PRT_DIS_P3})
- new net USBA2_OCS_N: R631.2
- new net USBA2_PWR_EN: R631.1, U601.58 (PF15)
- new net USBA2_SS_RXN: U601.33 (USB3DN_RXDM3)
- new net USBA2_SS_RXP: U601.32 (USB3DN_RXDP3)
- new net USBA2_SS_TXN: C608.2
- new net USBA2_SS_TXP: C607.2
- new net VBUS_LAPTOP: R625.1
- no-connect marks 0 -> 14
Other:
- note added: "(non-removable 1/4/6, BC on 2/3 only) when it is alive; with the RP2350 dead the strap defaults are safe."
- note added: "+1V15 bulk 4x22 uF sits at the TPS62933P (power_rails); route +1V15 as a pour on L4 under the hub."
- note added: "1. USB7206C USB 3.2 Gen2 hub, VQFN-100 12x12 (EP = VSS, via array to GND planes)"
- note added: "2. HUB TX AC-COUPLING 220 nF 0402 X7R in series with every hub SS TX (upstream + 5 downstream)."
- note added: "3. DECOUPLING VDD33 x8 pins, VCORE x9 pins: 100 nF per pin at the pin, plus 4.7 uF + 1 nF per rail (DS fig. 4-1)."
- note added: "4. CLOCK / BIAS / TEST / STRAPS"
- note added: "5. RESET / VBUS_DET / SMBUS"
- note added: "6. USB-A PORT POWER PRT_CTLx = combined power-enable output + overcurrent input (DS 8.2)"
- note added: "7. OPTIONAL SPI FLASH (DNP) only for Microchip-supplied custom firmware; ROM + straps + SMBus/OTP is the plan"
- note added: "8. PORT MAP (logical = physical on USB7206C) hub side (chip rotated with pins 76-100 toward the back edge)"
- note added: "CFG_NON_REM 200k PU = port 1 non-removable; CFG_BC_EN 10k PU = BC1.2 on ports 1-3. RP2350 refines both over SMBus"
- note added: "Embedded ports (1 GL3224, 4 RTL8156, 5 TUSB1046/PMG1, 6 RP2350): PRT_CTL floats (internal pull-up, never reads OC)."
- note added: "Firmware: SMB_PU high -> RESET_N low >= 5 us -> release -> wait >= 40 ms -> config -> AA56h. No other pull-ups on this bus."
- note added: "Hub RX pairs have no caps here: the transmitting chip's side (TUSB1064/TUSB1046/GL3224/RTL8156/USB-A sheet) provides them."
- note added: "Hub boots from flash only if it holds a valid image with the '2DFU' signature at 0x3FFFA; a blank flash -> ROM boot."
- note added: "Hub held in standby until +1V15 is in regulation (implies +3V3 up); 10k pull-up then releases it. trst >= 5 us."
- note added: "P1 : GL3224 card reader left side, upper CR_* (non-removable, strap)"
- note added: "P2 : USB-A #1 left side, lower USBA1_* (BC1.2, PRT_CTL2)"
- note added: "P3 : USB-A #2 bottom side, left USBA2_* (BC1.2, PRT_CTL3)"
- note added: "P4 : RTL8156BG 2.5GbE bottom side, right ETH_* (route around the PF/right side to the back-right)"
- note added: "P5 : TUSB1046 downstream C top side, right HUB_DSC_*"
- note added: "P6 : RP2350 (USB2 only) bottom-right corner MCU_USB_DP/DN (USB2 can use an inner layer to reach the MCU)"
- note added: "PF3-7 (I2S), PF18/31 (I2C master), PF19 (MIC_DET), PF29 (GPIO93): unused -> 100k PD. PF8/9 NC. PRT_CTL1/4/5/6 float."
- note added: "Place caps within ~5 mm of the hub pins, symmetric per pair, cut the reference plane under the 0402 pads (L2 void) for 10G."
- note added: "RESET_N = HUB_RESET_N (RP2350 open-drain) AND RAILS_PG (TPS62933P PG, open drain, 100k on power_rails) via D601."
- note added: "SMBus slave addr 0x2D. Pull-ups only when HUB_SMB_PU (RP2350 GPIO) is high -> hub enters CFG_SMBUS and waits for"
- note added: "Straps are latched at POR / RESET_N rising edge (hold >= 1 ms after). Config 3 (STRAP2 200k PD, STRAP1 10k PD) is the"
- note added: "UP : laptop via TUSB1064 top side, center HUB_UP_SS_*, LAPTOP_USB_DP/DN"
- note added: "USB-A #1 = hub port 2 (PRT_CTL2, PF16), USB-A #2 = hub port 3 (PRT_CTL3, PF15). Port on: pin = input + internal ~50k"
- note added: "USBAx_PWR_EN and USBAx_OCS_N are therefore the SAME node (0R ties, R630/R631). Do NOT add an external pull-up."
- note added: "VBUS_DET (PF30): laptop VBUS / 2 (47k/47k), BAT54WS clamp to +3V3: 4.4 V -> 2.2 V (VIH 2.1), 5.25 V -> 2.63 V (<2.7 V"
- note added: "VBUS_DET = 0 (no laptop): BC1.2 ports run as DCP; VBUS_DET = 1: CDP once the host powers the port."
- note added: "VCORE ~1.31 A (10G upstream + 5x 10G ports: 410 + 5*179 mA), VDD33 ~0.09 A -> ~1.8 W total; theta-JA 19 C/W (2S2P) -> ~+35 K."
- note added: "With the flash fitted the CE#/D0 strap resistors stay (they are read before the flash is probed). Fit R614 (D3 10k PU)"
- note added: "and remove R613 (D3 PD) so HOLD# is inactive. Flash images come only from Microchip -> not planned for odeck-10."
- note added: "no pull-ups seen -> hub boots from ROM+straps+OTP immediately -> RP2350 BOOTSEL (UF2) still enumerates on port 6."
- note added: "only valid USB7206C mode: PF26/27 = SMBus slave, PF15/16 = PRT_CTL3/2, PF30 = VBUS_DET, PF18/31 = I2C master (unused)."
- note added: "per checklist), 28 V -> ~3.6 V clamp. VBUS present = laptop attached (deck sources VBUS only after attach)."
- note added: "pull-up (EN high), switch FAULT# (open drain) pulls it low = overcurrent; port off: hub drives it low."
- note added: "the RP2350's config + USB_ATTACH_WITH_SMBUS (AA56h). HUB_SMB_PU low/floating (RP2350 off, BOOTSEL, broken FW):"
- note added: "usb_a sheet: TPS2553 EN = PWR_EN OR FORCE_EN (gate input, high-Z), FAULT# open-drain -> OCS_N."
- note removed: "TODO — planned contents: Microchip USB7206C: up=TUSB1064 USB, 10G ports -> USB-A x2, downstream C, GL3224, RTL8156BG; USB2 port -> RP2350. SMBus 0x2D to RP2350 (pull-ups powered by RP2350 GPIO), reset from RP2350."
- title: odeck-10 — USB hub -> odeck-10 — USB 3.2 Gen2 hub (USB7206C)

Commit message: Schematic review + footprint verification; fix all MAJOR findings
Reviews (docs/review/): power, PD/mux, data path, MCU/UI - 0 blockers,
7 majors, all resolved:
- power: diode-OR inputs (no shutdown-based PD-in priority), sink hand-over
  gated by delayed PG_5V, PD-in capacitance within 100 uF, HV resistor sizes,
  OVP filter/threshold, VBB_PG soft-start qualification
- card reader MS2_INS/SD2_WP phantom card, hub VBUS_DET level buffer
- RP2350 inductor dot text; minors across all sheets (HPD pull-down, PMG1
  INT pin, PHY TX caps, erratum E9 pull-downs, PHY I2C bridge gating,
  backlight 39 ohm, +1V1 cap, IOX P7)
Footprints: all 54 custom footprints checked vs manufacturer drawings,
50 fixed (courtyards, pads, paste, RJ45 mirrored pinout, EP sizes, holes);
removed obsolete FL_001 placeholder.
Firmware rules collected in docs/design/mcu.md.
186 parts, all JLC stock >= 5; netlist verify OK; ERC clean.

Co-Authored-By: Claude Opus 5.5 <noreply@anthropic.com>
Parts:
- added C641: 100n, Capacitor_SMD:C_0402_1005Metric, symbol Device:C
- added R632: 15k, Resistor_SMD:R_0402_1005Metric, symbol Device:R
- added R633: 49.9k, Resistor_SMD:R_0402_1005Metric, symbol Device:R
- added U603: 74LVC1G17, Package_TO_SOT_SMD:SOT-23-5, symbol 74xGxx:74LVC1G17
- R626: value 47k -> 68k; LCSC C25792 -> C36871
- R629: value 100k -> 4.7k; LCSC C25741 -> C25900
Connections:
- net +3V3: now also C641.1, U603.5 (VCC)
- net GND: now also C641.2, R633.2, U603.3 (GND)
- net HUB_VBUS_DET: now also R632.2, R633.1; no longer D602.2 (A), R625.2, R626.1
- new net HUB_VBUS_BUF: R632.1, U603.4
- new net HUB_VBUS_SNS: D602.2 (A), R625.2, R626.1, U603.2
- no-connect marks 14 -> 15
Other:
- note added: "(<= 2.7 V checklist 5.1, > VIH 2.1 V); 11k/49.9k from the checklist would give 2.73 V at our 3.33 V rail -> 15k."
- note added: "5.5 V-tolerant input) -> 15k/49.9k -> PF30. Sense node: 4.4 V -> 2.60 V (> VT+ max 2.0 V), 28 V -> ~3.6 V clamp (OK for"
- note added: "Buffer powered from +3V3 = same rail as VDD33 -> VBUS_DET can never rise before VDD33."
- note added: "VBUS present = laptop attached (deck sources VBUS only after attach). Limitation (review data #6): VBUS also exists for"
- note added: "VBUS_DET (PF30): VBUS_LAPTOP -> 47k/68k (x0.591) + BAT54WS clamp to +3V3 -> HUB_VBUS_SNS -> 74LVC1G17 (+3V3, Schmitt,"
- note added: "a powered-off laptop / charge-only cable -> hub waits as CDP, USB-A get no VBUS until FORCE_EN (firmware)."
- note added: "the LVC input), vSafe0V 0.8 V -> 0.47 V (< VT- min 0.8 V). PF30 high = +3V3 x 0.769 = 2.46-2.64 V for +3V3 3.20-3.43 V"
- note removed: "VBUS_DET (PF30): laptop VBUS / 2 (47k/47k), BAT54WS clamp to +3V3: 4.4 V -> 2.2 V (VIH 2.1), 5.25 V -> 2.63 V (<2.7 V"
- note removed: "per checklist), 28 V -> ~3.6 V clamp. VBUS present = laptop attached (deck sources VBUS only after attach)."

Commit message: Cost pass, PCB sync + rough placement, renders, README
- cost pass: extended parts 129 -> 114 (~$45/order less), nets unchanged
- tools/pcbsync.py: scripted update-PCB-from-schematic (keeps placed parts)
- tools/set_outline.py; board grown to 130x85 mm (provisional)
- hardware/odeck-10/placement.py: edge connectors + anchor-based packing,
  small passives spill to bottom; all 796 parts on the board (2 at anchor)
- docs/images: top/bottom/iso renders of the rough placement
- README.md: overview, architecture, repo layout, workflow, roadmap

Co-Authored-By: Claude Opus 5.5 <noreply@anthropic.com>
Parts:
- R626: footprint Resistor_SMD:R_0402_1005Metric -> Resistor_SMD:R_0603_1608Metric; LCSC C36871 -> C23231
- R633: footprint Resistor_SMD:R_0402_1005Metric -> Resistor_SMD:R_0603_1608Metric; LCSC C25897 -> C23184
Changed lines of the file:
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@@
 			)
 		)
-		(property "Footprint" "Resistor_SMD:R_0402_1005Metric"
+		(property "Footprint" "Resistor_SMD:R_0603_1608Metric"
 			(at 353.06 167.64 0)
 			(effects
@@
 			)
 		)
-		(property "LCSC" "C36871"
+		(property "LCSC" "C23231"
 			(at 353.06 167.64 0)
 			(effects
@@
 			)
 		)
-		(property "Footprint" "Resistor_SMD:R_0402_1005Metric"
+		(property "Footprint" "Resistor_SMD:R_0603_1608Metric"
 			(at 454.66 167.64 0)
 			(effects
@@
 			)
 		)
-		(property "LCSC" "C25897"
+		(property "LCSC" "C23184"
 			(at 454.66 167.64 0)
 			(effects
