File: hardware/odeck-10/usbc_muxes.kicad_sch (KiCad schematic)
At the start: 0 parts

Commit message: Draft data-path sheets: PD controller, USB-C muxes/DP, USB hub
- pd_pmg1: PMG1-S3 (CYPM1321, dead-battery Rd) dual-port: laptop EPR source +
  DP UFP_D, downstream 5 V/3 A + DP DFP_D, HPD relay, VBUS-powered cold start,
  I2C 0x42, SWD/reset via cuttable jumpers
- usbc_muxes: laptop + downstream USB-C, TUSB1064/TUSB1046 in GPIO mode,
  TPD4S480 (EPR) / TPD6S300 CC protection, 10G-rated ESD, AC coupling
- usb_hub: USB7206C port map, SMBus-optional boot, reset gated by RAILS_PG,
  BC1.2 on USB-A ports, hub-TX AC caps
- schgen: in_bom option; nets: VBUS_LSW, PMG1_VDDD, hub/mux/CC links
- import_lcsc.sh: guard against overwriting other parts' footprints
- 137 parts, all JLC stock >= 5

Co-Authored-By: Claude Opus 5.5 <noreply@anthropic.com>
Parts:
- added C501, C536, C537: 100n/50V, Capacitor_SMD:C_0603_1608Metric, symbol Device:C
- added C502: 100n/100V, Capacitor_SMD:C_0603_1608Metric, symbol Device:C
- added C503, C538: 1u, Capacitor_SMD:C_0402_1005Metric, symbol Device:C
- added C504, C505, C506, C508, C523, C524, C525, C526, C527, C528: 100n, Capacitor_SMD:C_0402_1005Metric, symbol Device:C
- added C507, C529: 10u, Capacitor_SMD:C_0603_1608Metric, symbol Device:C
- added C509, C510, C511, C512, C513, C514, C515, C516, C517, C518, C519, C520, C521, C522, C530, C531, C532, C533, C534, C535: 220n, Capacitor_SMD:C_0402_1005Metric, symbol Device:C
- added D501: SMBJ30A, Diode_SMD:D_SMB, symbol Device:D_Zener
- added D502, D503, D504, D506, D507: TPD4E02B04, odeck:USON-10_L2.5-W1.0-P0.50-BL, symbol odeck:TPD4E02B04DQAR
- added D505: SMAJ6.0A, Diode_SMD:D_SMA, symbol Device:D_Zener
- added J501: USB-C laptop, odeck:USB-C-TH_DX07S024XJ1R1100-1, symbol odeck:DX07S024XJ1R1100
- added J502: USB-C downstream, odeck:USB-C-SMD_TYPE-C-24P, symbol odeck:12401610E4#2A
- added R501, R525, R526, R541: 100k, Resistor_SMD:R_0402_1005Metric, symbol Device:R
- added R502, R503, R542, R543: 2M, Resistor_SMD:R_0603_1608Metric, symbol Device:R
- added R504, R505, R522, R523, R524: 10k, Resistor_SMD:R_0402_1005Metric, symbol Device:R
- added R506, R507: 1M, Resistor_SMD:R_0402_1005Metric, symbol Device:R
- added R508, R509, R511, R513, R514, R515, R517, R519, R521, R527, R528, R530, R532, R533, R534, R536, R537, R538, R539, R540: 1k, Resistor_SMD:R_0402_1005Metric, symbol Device:R
- added R510, R512, R516, R518, R520, R529, R531, R535: 20k, Resistor_SMD:R_0402_1005Metric, symbol Device:R
- added U501: TPD4S480, odeck:WQFN-20_L3.0-W3.0-P0.40-BL-EP1.7, symbol odeck:TPD4S480RUKR_C43131250
- added U502: TUSB1064, odeck:WQFN-40_L6.0-W4.0-P0.40-TL-EP, symbol odeck:TUSB1064IRNQT
- added U503: TUSB1046-DCI, odeck:WQFN-40_L6.0-W4.0-P0.40-TL-EP, symbol odeck:TUSB1046-DCIRNQT
- added U504: TPD6S300, odeck:WQFN-20_L3.0-W3.0-P0.40-BL-EP1.7, symbol odeck:TPD6S300RUKR
Connections:
- new net +3V3: C504.1, C505.1, C506.1, C507.1, C525.1, C526.1, C527.1, C528.1, C529.1, C538.1, R504.2, R506.2, R509.2, R511.2, R513.2, R515.2, R517.2, R519.2, R521.2, R523.2, R526.2, R528.2, R530.2, R532.2, R534.2, R536.2, R538.2, R540.2, R541.2, U502.20 (VCC), U502.28 (VCC), U502.6 (VCC), U503.1 (VCC), U503.20 (VCC), U503.28 (VCC), U503.6 (VCC), U504.10 (VPWR)
- new net DP_AUX_N: C524.1, R507.1, U502.27 (AUXn)
- new net DP_AUX_P: C523.1, R506.1, U502.26 (AUXp)
- new net DP_ML0_N: C516.1, U502.39 (DP0n)
- new net DP_ML0_P: C515.1, U502.40 (DP0p)
- new net DP_ML1_N: C518.1, U502.36 (DP1n)
- new net DP_ML1_P: C517.1, U502.37 (DP1p)
- new net DP_ML2_N: C520.1, U502.33 (DP2n)
- new net DP_ML2_P: C519.1, U502.34 (DP2p)
- new net DP_ML3_N: C522.1, U502.30 (DP3n)
- new net DP_ML3_P: C521.1, U502.31 (DP3p)
- new net DS_AUX_N: C524.2, R526.1, U503.25 (AUXn)
- new net DS_AUX_P: C523.2, R525.1, U503.24 (AUXp)
- new net DS_CAD_SNK: R523.1, R524.1, U503.29 (CAD_SNK/RSVD1)
- new net DS_CC1: U504.12 (CC1)
- new net DS_CC2: U504.11 (CC2)
- new net DS_CCPROT_FLT_N: R541.1, U504.9 (~{FLT})
- new net DS_C_CC1: J502.A5 (CC1), U504.4 (C_CC1)
- new net DS_C_CC2: J502.B5 (CC2), U504.5 (C_CC2)
- new net DS_C_SBU1: J502.A8 (SBU1), U504.1 (C_SBU1)
- new net DS_C_SBU2: J502.B8 (SBU2), U504.2 (C_SBU2)
- new net DS_C_TX1_N: C533.2, D506.2 (IO2), D506.9 (NC), J502.A3 (SSTXn1)
- new net DS_C_TX1_P: C532.2, D506.1 (IO1), D506.10 (NC), J502.A2 (SSTXp1)
- new net DS_C_TX2_N: C535.2, D507.2 (IO2), D507.9 (NC), J502.B3 (SSTXn2)
- new net DS_C_TX2_P: C534.2, D507.1 (IO1), D507.10 (NC), J502.B2 (SSTXp2)
- new net DS_DPEQ0: R539.1, R540.1, U503.14 (DPEQ0/A1)
- new net DS_DPEQ1: R537.1, R538.1, U503.2 (DPEQ1)
- new net DS_DP_ML0_N: C516.2, U503.10 (DP0n)
- new net DS_DP_ML0_P: C515.2, U503.9 (DP0p)
- new net DS_DP_ML1_N: C518.2, U503.13 (DP1n)
- new net DS_DP_ML1_P: C517.2, U503.12 (DP1p)
- new net DS_DP_ML2_N: C520.2, U503.16 (DP2n)
- new net DS_DP_ML2_P: C519.2, U503.15 (DP2p)
- new net DS_DP_ML3_N: C522.2, U503.19 (DP3n)
- new net DS_DP_ML3_P: C521.2, U503.18 (DP3p)
- new net DS_EQ0: R531.1, R532.1, U503.38 (EQ0)
- new net DS_EQ1: R529.1, R530.1, U503.35 (EQ1)
- new net DS_HPD: R522.1
- new net DS_HPDIN: R522.2, U503.32 (HPDIN/RSVD2)
- new net DS_I2C_EN: R527.1, R528.1, U503.17 (I2C_EN)
- new net DS_RX1_N: D506.5 (IO4), D506.6 (NC), J502.B10 (SSRXn1), U503.31 (RX1n)
- new net DS_RX1_P: D506.4 (IO3), D506.7 (NC), J502.B11 (SSRXp1), U503.30 (RX1p)
- new net DS_RX2_N: D507.5 (IO4), D507.6 (NC), J502.A10 (SSRXn2), U503.39 (RX2n)
- new net DS_RX2_P: D507.4 (IO3), D507.7 (NC), J502.A11 (SSRXp2), U503.40 (RX2p)
- new net DS_SBU1: R542.1, U503.27 (SBU1), U504.15 (SBU1)
- new net DS_SBU2: R543.1, U503.26 (SBU2), U504.14 (SBU2)
- new net DS_SSEQ0: R535.1, R536.1, U503.11 (SSEQ0/A0)
- new net DS_SSEQ1: R533.1, R534.1, U503.3 (SSEQ1)
- new net DS_SSRX_N: C531.1, U503.4 (SSRXn)
- new net DS_SSRX_P: C530.1, U503.5 (SSRXp)
- new net DS_TPD_VBIAS: C537.1, U504.3 (VBIAS)
- new net DS_TX1_N: C533.1, U503.34 (TX1n)
- new net DS_TX1_P: C532.1, U503.33 (TX1p)
- new net DS_TX2_N: C535.1, U503.36 (TX2n)
- new net DS_TX2_P: C534.1, U503.37 (TX2p)
- new net GND: C501.2, C502.2, C503.2, C504.2, C505.2, C506.2, C507.2, C508.2, C525.2, C526.2, C527.2, C528.2, C529.2, C536.2, C537.2, C538.2, D501.2 (A), D502.3 (GND), D502.8 (GND), D503.3 (GND), D503.8 (GND), D504.3 (GND), D504.8 (GND), D505.2 (A), D506.3 (GND), D506.8 (GND), D507.3 (GND), D507.8 (GND), J501.0, J501.A1 (GND), J501.A12 (GND), J501.B1 (GND), J501.B12 (GND), J502.14 (SHEELD), J502.15 (SHEELD), J502.A1 (GND), J502.A12 (GND), J502.B1 (GND), J502.B12 (GND), R502.2, R503.2, R507.2, R508.2, R510.2, R512.2, R514.2, R516.2, R518.2, R520.2, R524.2, R525.2, R527.2, R529.2, R531.2, R533.2, R535.2, R537.2, R539.2, R542.2, R543.2, U501.13 (GND), U501.18 (GND), U501.21 (EP), U501.8 (GND), U502.41 (EP), U503.41 (EP), U504.13 (GND), U504.16 (N.C.), U504.17 (N.C.), U504.18 (GND), U504.21 (EP), U504.6 (RPD_G2), U504.7 (RPD_G1), U504.8 (GND)
- new net HUB_DSC_DN: J502.A7 (Dn1), J502.B7 (Dn2), U504.19 (D2)
- new net HUB_DSC_DP: J502.A6 (Dp1), J502.B6 (Dp2), U504.20 (D1)
- new net HUB_DSC_SS_RXN: C531.2
- new net HUB_DSC_SS_RXP: C530.2
- new net HUB_DSC_SS_TXN: U503.7 (SSTXn)
- new net HUB_DSC_SS_TXP: U503.8 (SSTXp)
- new net HUB_UP_SS_RXN: C514.2
- new net HUB_UP_SS_RXP: C513.2
- new net HUB_UP_SS_TXN: U502.7 (SSTXn)
- new net HUB_UP_SS_TXP: U502.8 (SSTXp)
- new net LAPTOP_CC1: U501.12 (CC1)
- new net LAPTOP_CC2: U501.11 (CC2)
- new net LAPTOP_USB_DN: D504.2 (IO2), D504.9 (NC), J501.A7 (DN1), J501.B7 (DN2)
- new net LAPTOP_USB_DP: D504.1 (IO1), D504.10 (NC), J501.A6 (DP1), J501.B6 (DP2)
- new net MUX_DS_CTL0: U503.22 (CTL0/SDA)
- new net MUX_DS_CTL1: U503.23 (CTL1/HPDIN)
- new net MUX_DS_FLIP: U503.21 (FLIP/SCL)
- new net MUX_UP_CTL0: U502.22 (CTL0/SDA)
- new net MUX_UP_CTL1: U502.23 (CTL1)
- new net MUX_UP_FLIP: U502.21 (FLIP/SCL)
- new net PMG1_VDDD: C503.1, R501.2, U501.10 (VPWR), U501.16 (EPR_EN)
- new net UP_CCPROT_FLT_N: R501.1, U501.9 (~{FLT})
- new net UP_C_CC1: J501.A5 (CC1), U501.4 (C_CC1), U501.7 (RPD_G1)
- new net UP_C_CC2: J501.B5 (CC2), U501.5 (C_CC2), U501.6 (RPD_G2)
- new net UP_C_SBU1: J501.A8 (SUB1), U501.1 (C_SBU1)
- new net UP_C_SBU2: J501.B8 (SUB2), U501.2 (C_SBU2)
- new net UP_C_TX1_N: C510.2, D502.2 (IO2), D502.9 (NC), J501.A3 (SSTXn1)
- new net UP_C_TX1_P: C509.2, D502.1 (IO1), D502.10 (NC), J501.A2 (SSTXP1)
- new net UP_C_TX2_N: C512.2, D503.2 (IO2), D503.9 (NC), J501.B3 (SSTXn2)
- new net UP_C_TX2_P: C511.2, D503.1 (IO1), D503.10 (NC), J501.B2 (SSTXp2)
- new net UP_DPEQ0: R520.1, R521.1, U502.35 (DPEQ0/A1)
- new net UP_DPEQ1: R518.1, R519.1, U502.2 (DPEQ1)
- new net UP_EQ0: R512.1, R513.1, U502.11 (EQ0)
- new net UP_EQ1: R510.1, R511.1, U502.14 (EQ1)
- new net UP_HPD: R505.1
- new net UP_HPDIN: R505.2, U502.32 (HPDIN)
- new net UP_I2C_EN: R508.1, R509.1, U502.17 (I2C_EN)
- new net UP_MUX_EN: C508.1, R504.1, U502.29 (EN)
- new net UP_RX1_N: D502.5 (IO4), D502.6 (NC), J501.B10 (SSRXn1), U502.13 (RX1n)
- new net UP_RX1_P: D502.4 (IO3), D502.7 (NC), J501.B11 (SSRXp1), U502.12 (RX1p)
- new net UP_RX2_N: D503.5 (IO4), D503.6 (NC), J501.A10 (SSRXn2), U502.15 (RX2n)
- new net UP_RX2_P: D503.4 (IO3), D503.7 (NC), J501.A11 (SSRXp2), U502.16 (RX2p)
- new net UP_SBU1: R502.1, U501.15 (SBU1), U502.24 (SBU1)
- new net UP_SBU2: R503.1, U501.14 (SBU2), U502.25 (SBU2)
- new net UP_SSEQ0: R516.1, R517.1, U502.38 (SSEQ0/A0)
- new net UP_SSEQ1: R514.1, R515.1, U502.3 (SSEQ1)
- new net UP_SSRX_N: C514.1, U502.4 (SSRXn)
- new net UP_SSRX_P: C513.1, U502.5 (SSRXp)
- new net UP_TPD_VBIAS: C502.1, U501.3 (VBIAS)
- new net UP_TX1_N: C510.1, U502.10 (TX1n)
- new net UP_TX1_P: C509.1, U502.9 (TX1p)
- new net UP_TX2_N: C512.1, U502.18 (TX2n)
- new net UP_TX2_P: C511.1, U502.19 (TX2p)
- new net VBUS_DS: C536.1, D505.1 (K), J502.A4 (VBUS), J502.A9 (VBUS), J502.B4 (VBUS), J502.B9 (VBUS)
- new net VBUS_LAPTOP: C501.1, D501.1 (K), J501.A4 (VBUS), J501.A9 (VBUS), J501.B4 (VBUS), J501.B9 (VBUS), U501.20 (VBUS)
- no-connect marks 0 -> 7
Other:
- note added: "-> TUSB1046 HPDIN."
- note added: "1. LAPTOP USB-C (UFP data, EPR source up to 28 V x 5 A, bus-powered sink 5 V)"
- note added: "2. TUSB1064 UFP_D MUX/REDRIVER (TUSB1064IRNQT C702365, GPIO mode: I2C_EN = 0)"
- note added: "3. DP MAIN LINK + AUX TUSB1064 -> TUSB1046 (one cap per line, both redrivers are linear: transparent to link training)"
- note added: "4. TUSB1046-DCI DFP_D MUX/REDRIVER (TUSB1046-DCIRNQT C2652434, GPIO mode: I2C_EN = 0)"
- note added: "5. DOWNSTREAM USB-C (DFP data, 5 V / 3 A source by PMG1 port 1, DP alt mode DFP_D)"
- note added: "500k internal pull-down). CTL1/CTL0: LL power down | LH USB3 only | HL 4-lane DP (pin assign. C) | HH USB3 + 2-lane DP (D)."
- note added: "6. INTERFACES / ASSUMPTIONS"
- note added: "A2/A3 TX1+/- B2/B3 TX2+/- (ours: TUSB1064 TX through 220 nF) B11/B10 RX1+/- A11/A10 RX2+/- (DC to TUSB1064 RX)"
- note added: "A6/B6 D+ and A7/B7 D- tied at the connector -> LAPTOP_USB_DP/DN (hub upstream USB2). A8/B8 SBU1/2 -> TPD4S480."
- note added: "AC coupling: 220 nF on our TX1/TX2 (to receptacle TX pins) and on SSRX -> HUB_UP_SS_RX (we transmit into the hub)."
- note added: "AUX: AUXp 100k -> GND, AUXn 100k -> +3V3 (DFP_D/source bias seen by the monitor). SBU1/2 via TPD6S300, 2M to GND."
- note added: "AUX: AUXp 1M -> +3V3, AUXn 1M -> GND (UFP_D/sink bias seen by the laptop), 100 nF to TUSB1046 AUX (section 4)."
- note added: "AUX: one 100 nF per line between the two bias networks (TUSB1064 side 1M up/down, TUSB1046 side 100k down/up)."
- note added: "Amphenol 12401610E4#2A (C5119948): 20 V / 5 A, USB 3.2 Gen2. Shield pins 14/15 -> GND."
- note added: "CC FETs pass VCONN (600 mA) if PMG1 port 1 supplies it. FLT# -> DS_CCPROT_FLT_N (100k to +3V3), optional PMG1 GPIO."
- note added: "CC lines: cReceiver caps (PMG1 reference 390 pF) and VCONN source belong to pd_pmg1 next to the PMG1 CC pins."
- note added: "CTL1/CTL0: LL power down | LH USB3 only | HL 4-lane DP (C/E) | HH USB3 + 2-lane DP (D/F). Default after power-up: USB3."
- note added: "Controlled by PMG1 port 0: MUX_UP_CTL1 = DP enabled, MUX_UP_CTL0 = USB3 enabled, MUX_UP_FLIP = plug flipped (all fail-safe,"
- note added: "Controlled by PMG1 port 1: MUX_DS_CTL1 = DP enabled, MUX_DS_CTL0 = USB3 enabled, MUX_DS_FLIP = plug flipped."
- note added: "DP0..DP3 220 nF (75-265 nF). 2 lanes used in pin assignment D (laptop advertises D: USB3 stays up), all 4 in C."
- note added: "DPEQ1/DPEQ0 = 0/0 #0 1.0 dB (from TUSB1064 over ~30 mm)."
- note added: "DPEQ1/DPEQ0 = R/R #5 6.5 dB at 4.05 GHz (laptop cable, DP lanes)"
- note added: "DS_HPD = downstream monitor HPD as decoded by PMG1 port 1 (DFP_D) from DP Status / Attention VDMs (incl. IRQ_HPD pulses)"
- note added: "EN: 10k/100n RC to +3V3 -> 4-level pins latched ~1 ms after VCC. HPDIN <- UP_HPD (10k series: pin not fail-safe)."
- note added: "EPR_EN = VPWR (divider always on, keeps unloaded VBUS_LV < 24 V abs max); VBUS_LV, EPR_BLK_G open (PMG1 senses 28 V)."
- note added: "EQ straps (bench-tunable, both footprints on every 4-level pin):"
- note added: "EQ straps: EQ1/EQ0 = R/1 #7 5.2 dB (downstream cable -> RX1/RX2) SSEQ1/SSEQ0 = 0/F #2 1.7 dB (hub TX, short)"
- note added: "EQ1/EQ0 = R/F #6 6.6 dB (laptop cable -> RX1/RX2, USB) SSEQ1/SSEQ0 = 0/1 #3 2.2 dB (hub TX, ~40 mm)"
- note added: "ESD TPD4E02B04 on all 8 SS lines, flow-through at the connector."
- note added: "ESD: TPD4E02B04 (0.25 pF, 10 Gbps) on all 8 SS lines + USB2, at the connector, flow-through (route over pads 1-10, 2-9, 4-7, 5-6)."
- note added: "FETs stay open and the laptop sees only the dead-battery Rd. RPD_Gx = C_CCx: dead-battery Rd while VPWR is off, so a"
- note added: "FLT# (open drain) -> UP_CCPROT_FLT_N, pulled up to PMG1_VDDD; route to a PMG1 GPIO if pins allow (optional)."
- note added: "HPD (both nets are PMG1 OUTPUTS on pd_pmg1 and mux HPDIN INPUTS here; 10k series, internal 500k pull-downs):"
- note added: "HPDIN (pin 32 in GPIO mode) <- DS_HPD through 10k (pin not fail-safe). CAD_SNK = H (10k to +3V3): AUX snoop off,"
- note added: "HUB_UP_SS_TX -> SSTX is DC here: the 220 nF hub-TX caps sit on usb_hub. RX1/RX2 DC (the laptop TX has its caps)."
- note added: "Hub links: hub-TX 220 nF caps on usb_hub, hub-RX 220 nF caps (our SSRX outputs) on this sheet."
- note added: "I2C: both muxes in GPIO mode, SDA/SCL pins are CTL0/FLIP; I2C_EN pull-up footprints (DNP) for a later I2C variant."
- note added: "In GPIO mode AUX snoop is off: all DP lanes of the selected config are on while HPDIN is high; off after HPDIN low > 2 ms."
- note added: "JAE DX07S024XJ1R1100 (C134113): 48 V / 5 A, USB 3.x 10G. Shell -> GND (direct, JLC practice; via-stitch to plane)."
- note added: "OVP (power_laptop) trips at ~30.8 V, LM74800 backstop 32.6 V. Only 100 nF on VBUS here (cSnkBulk budget on power_laptop)."
- note added: "PMG1_VDDD (global, pd_pmg1): powers TPD4S480 VPWR (~0.16 mA) so CC works in a dead deck. Optional new nets kept local:"
- note added: "Pins by number (A row / B row checked vs USB Type-C R2.x receptacle table and symbol names):"
- note added: "Power-up default is USB3 mode: PMG1 must pulse CTL0 L-H-L to power it down when nothing is attached. 16 ms debounce."
- note added: "Pull-downs: internal 500k in both muxes -> lanes off while PMG1 is in reset."
- note added: "RPD_G1/2 = GND: NO dead-battery Rd on a source-only port. N.C. pins 16/17 -> GND per datasheet."
- note added: "Route as 85 ohm diff (90 ohm AUX), DP lanes length-matched within a pair (<0.1 mm), between pairs < 2 mm. Keep < 50 mm."
- note added: "Rule: exactly one 75-265 nF cap per SS line, at the transmitter end of each segment."
- note added: "SBU1/2 DC to the receptacle via TPD4S480, 2M to GND. I2C option: fit the 1k I2C_EN pull-up and re-wire CTL0/FLIP as SDA/SCL."
- note added: "TPD4S480 (C43131250): 63 V short-to-VBUS OVP + IEC ESD on CC1/CC2/SBU1/SBU2 (PMG1 CC/SBU pins are 6 V abs max)."
- note added: "TPD6S300 (C2649810): 24 V CC/SBU OVP + IEC ESD (CC, SBU, D+/D-); VPWR = +3V3 (port 1 only runs with the deck powered)."
- note added: "TUSB1064 DP lanes; low > 2 ms turns them off, IRQ_HPD pulses are harmless)."
- note added: "TVS SMAJ6.0A on VBUS_DS (6 V standoff over 5.25 V max). 100 nF at the connector."
- note added: "UP_CCPROT_FLT_N / DS_CCPROT_FLT_N. DP_ML0/1 and DP_AUX nets are global names but only used on this sheet."
- note added: "UP_HPD = HPD state PMG1 port 0 (UFP_D) reports to the laptop (DP Status/Attention) -> TUSB1064 HPDIN (enables the"
- note added: "USB side: HUB_DSC_SS_TX -> SSTX DC (hub-TX caps on usb_hub); SSRX -> 220 nF -> HUB_DSC_SS_RX. Receptacle TX via 220 nF, RX DC."
- note added: "USB2 D+/D- (both rows) -> HUB_DSC_DP/DN directly (ESD in TPD6S300 D1/D2). VBUS_DS switch + bulk cap: pd_pmg1 / power."
- note added: "VBUS TVS SMBJ30A: VRWM 30 V > 29.4 V (28 V EPR +5 %), VBR 33.3 V min, below PMG1 VBUS abs max 34 V at low current;"
- note added: "VPWR = PMG1_VDDD: the PMG1 always-on rail (from VBUS or the deck). It MUST be up whenever PMG1 runs, otherwise the CC"
- note added: "lanes follow CTL only (robust with non-compliant AUX); DNP pull-down re-enables snoop (lane power saving)."
- note added: "laptop applies 5 V to a dead deck (bus-powered cold start). Removed 3.5 ms after VPWR is up -> PMG1 owns CC (Rp/Rd/DRP)."
- note removed: "TODO — planned contents: Laptop USB-C (JAE DX07S024XJ1R1100) + TUSB1064 (UFP), downstream USB-C (Amphenol 12401610E4#2A) + TUSB1046-DCI (DFP), DP 2-lane HBR3 + AUX between muxes, ESD."
- title: odeck-10 — USB-C muxes & DP -> odeck-10 — USB-C ports, TUSB1064 / TUSB1046 alt-mode muxes

Commit message: Schematic review + footprint verification; fix all MAJOR findings
Reviews (docs/review/): power, PD/mux, data path, MCU/UI - 0 blockers,
7 majors, all resolved:
- power: diode-OR inputs (no shutdown-based PD-in priority), sink hand-over
  gated by delayed PG_5V, PD-in capacitance within 100 uF, HV resistor sizes,
  OVP filter/threshold, VBB_PG soft-start qualification
- card reader MS2_INS/SD2_WP phantom card, hub VBUS_DET level buffer
- RP2350 inductor dot text; minors across all sheets (HPD pull-down, PMG1
  INT pin, PHY TX caps, erratum E9 pull-downs, PHY I2C bridge gating,
  backlight 39 ohm, +1V1 cap, IOX P7)
Footprints: all 54 custom footprints checked vs manufacturer drawings,
50 fixed (courtyards, pads, paste, RJ45 mirrored pinout, EP sizes, holes);
removed obsolete FL_001 placeholder.
Firmware rules collected in docs/design/mcu.md.
186 parts, all JLC stock >= 5; netlist verify OK; ERC clean.

Co-Authored-By: Claude Opus 5.5 <noreply@anthropic.com>
Parts:
- added R544: 100k, Resistor_SMD:R_0402_1005Metric, symbol Device:R
- D501: value SMBJ30A -> SMCJ28A; footprint Diode_SMD:D_SMB -> Diode_SMD:D_SMC; LCSC C113998 -> C224047
Connections:
- net GND: now also R544.2
- net UP_HPD: now also R544.1
Other:
- note added: "(R(ENPD)). Both HPDIN inputs are therefore low while PMG1 is in reset -> lanes off."
- note added: "HPD (both nets are PMG1 OUTPUTS on pd_pmg1 and mux HPDIN INPUTS here; 10k series):"
- note added: "OVP latch (power_laptop, ~30.8 V) and the LM74800 backstop (32.6 V). Keep the VBUS caps close to J501 (hot-plug)."
- note added: "Only 100 nF on VBUS here (cSnkBulk budget on power_laptop)."
- note added: "Pull-downs: TUSB1064 HPDIN has none internally -> external 100k on UP_HPD; TUSB1046-DCI HPDIN has 150k internal"
- note added: "SMC over SMBJ: ~2.5x lower dynamic resistance -> lower clamp at a given surge current. Steady state is covered by the"
- note added: "TUSB1064 HPDIN has NO internal pull-down (DS p.6: 500k only on CTL0/CTL1/FLIP/EN): 100k UP_HPD -> GND here."
- note added: "VBUS TVS SMCJ28A (1500 W SMC): VRWM 28 V, VBR 31.1-34.4 V @1 mA, VC 45.4 V @33 A. At 29.4 V (28 V EPR +5 %) it is ~2 V"
- note added: "below VBR min -> leakage stays in the uA range (bench-check hot). It does NOT hold the PMG1 34 V abs-max pins below 34 V"
- note added: "during a surge (no TVS with VRWM >= 28 V can): accepted residual risk, same as Infineon's EPR references (VBUS_C direct)."
- note removed: "HPD (both nets are PMG1 OUTPUTS on pd_pmg1 and mux HPDIN INPUTS here; 10k series, internal 500k pull-downs):"
- note removed: "OVP (power_laptop) trips at ~30.8 V, LM74800 backstop 32.6 V. Only 100 nF on VBUS here (cSnkBulk budget on power_laptop)."
- note removed: "Pull-downs: internal 500k in both muxes -> lanes off while PMG1 is in reset."
- note removed: "VBUS TVS SMBJ30A: VRWM 30 V > 29.4 V (28 V EPR +5 %), VBR 33.3 V min, below PMG1 VBUS abs max 34 V at low current;"

Commit message: Cost pass, PCB sync + rough placement, renders, README
- cost pass: extended parts 129 -> 114 (~$45/order less), nets unchanged
- tools/pcbsync.py: scripted update-PCB-from-schematic (keeps placed parts)
- tools/set_outline.py; board grown to 130x85 mm (provisional)
- hardware/odeck-10/placement.py: edge connectors + anchor-based packing,
  small passives spill to bottom; all 796 parts on the board (2 at anchor)
- docs/images: top/bottom/iso renders of the rough placement
- README.md: overview, architecture, repo layout, workflow, roadmap

Co-Authored-By: Claude Opus 5.5 <noreply@anthropic.com>
Parts:
- C502: footprint Capacitor_SMD:C_0603_1608Metric -> Capacitor_SMD:C_0805_2012Metric; LCSC C15725 -> C28233
Changed lines of the file:
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@@
 			)
 		)
-		(property "Footprint" "Capacitor_SMD:C_0603_1608Metric"
+		(property "Footprint" "Capacitor_SMD:C_0805_2012Metric"
 			(at 93.98 152.40 0)
 			(effects
@@
 			)
 		)
-		(property "LCSC" "C15725"
+		(property "LCSC" "C28233"
 			(at 93.98 152.40 0)
 			(effects
