File: hardware/odeck-10/card_reader.kicad_sch (KiCad schematic)
At the start: 0 parts

Commit message: Draft remaining sheets: USB-A, card reader, Ethernet, MCU, display/UI, sensors
- usb_a: 2x 10G USB-A, TPS2553 switches (hub OR RP2350 force), INA180 sense
- card_reader: GL3224 + SD/microSD, card detect + activity to MCU
- ethernet: RTL8156BG with switched 3.3 V, 0.95 V PWM buck, 2.5G magjack,
  LED buffer, EUI-48 EEPROM + gated I2C bridge for MAC eFuse write
- mcu: RP2350B reference core, full GPIO table, TCA9534 expander, PIO I2C
- display_ui: 2.0" ST7789 LCD + backlight PWM, buttons, unpopulated GPIO
  header (series R + ESD), Qwiic
- sensors: 8x TMP1075, 2 NTCs, thermocouple pads
- integration: ETH_I2C_EN net, TPS62933F for +3V3, PWR_FLAGs
- schgen: deterministic UUIDs; bom_check: cost summary
- 181 parts, all JLC stock >= 5; netlist verify OK; ERC clean but 1 spare pin

Co-Authored-By: Claude Opus 5.5 <noreply@anthropic.com>
Parts:
- added C901: 10u, Capacitor_SMD:C_0805_2012Metric, symbol Device:C
- added C902, C905, C906, C907, C908, C914, C916, C917, C918: 100n, Capacitor_SMD:C_0402_1005Metric, symbol Device:C
- added C903: 10u, Capacitor_SMD:C_0603_1608Metric, symbol Device:C
- added C904, C910, C911, C912: 1u, Capacitor_SMD:C_0402_1005Metric, symbol Device:C
- added C909: 2.2u, Capacitor_SMD:C_0402_1005Metric, symbol Device:C
- added C913, C915: 4.7u, Capacitor_SMD:C_0402_1005Metric, symbol Device:C
- added C919, C920: 20p, Capacitor_SMD:C_0402_1005Metric, symbol Device:C
- added D901: green, LED_SMD:LED_0805_2012Metric, symbol Device:LED
- added J901: SD-111, odeck:SD-SMD_SD-111, symbol odeck:SD-111
- added J902: DM3AT, odeck:SD-SMD_DM3AT-SF-PEJM5, symbol odeck:DM3AT-SF-PEJM5
- added R901: 680, Resistor_SMD:R_0402_1005Metric, symbol Device:R
- added R902, R903: 10k, Resistor_SMD:R_0402_1005Metric, symbol Device:R
- added R904, R905, R906, R907: 1k, Resistor_SMD:R_0402_1005Metric, symbol Device:R
- added U901: GL3224-ONY04, odeck:QFN-48_L7.0-W7.0-P0.50-BL-EP5.1, symbol odeck:GL3224-ONY04
- added Y901: 25MHz, Crystal:Crystal_SMD_3225-4Pin_3.2x2.5mm, symbol Device:Crystal_GND24
Connections:
- new net +5V: C901.1, C902.1, U901.22 (VBUS)
- new net CR_1V2: C909.1, C910.1, U901.26 (DVDD12), U901.9 (AVDD12)
- new net CR_3V3: C903.1, C904.1, C905.1, C906.1, C907.1, C908.1, R902.2, U901.15 (AVDD33), U901.25 (DVDD33), U901.34 (DVDD33), U901.44 (DVDD33), U901.6 (AVDD33)
- new net CR_CD_SD_N: R904.2
- new net CR_CD_USD_N: R905.2
- new net CR_DN: U901.4 (DM)
- new net CR_DP: U901.5 (DP)
- new net CR_LED: R906.2
- new net CR_LED_A: D901.2 (A), R907.2
- new net CR_LED_IC: R906.1, R907.1, U901.21 (LED)
- new net CR_RTERM: R901.1, U901.16 (RTERM)
- new net CR_SD_CDZ: J901.10 (CD), R904.1, U901.1 (SD1_CDZ)
- new net CR_SD_CLK: J901.5 (CLK), U901.39 (S1CK_M1D0)
- new net CR_SD_CMD: J901.2 (CMD), U901.40 (S1CM_M1D2)
- new net CR_SD_D0: J901.7 (DAT0), U901.38 (S1D0_M1D1)
- new net CR_SD_D1: J901.8 (DAT1), U901.37 (S1D1_M1BS)
- new net CR_SD_D2: J901.9 (DAT2), U901.42 (S1D2_M1CK)
- new net CR_SD_D3: J901.1 (CD/DAT3), U901.41 (S1D3_M1D3)
- new net CR_SD_VCC: C913.1, C914.1, J901.4 (VDD), U901.23 (S1M1_VCC)
- new net CR_SD_WP: J901.11 (WP), U901.2 (MS1_INS/SD1_WP)
- new net CR_SPI_CK: R903.1, U901.19 (SPI_CK)
- new net CR_SPI_MISO: R902.1, U901.17 (SPI_MISO)
- new net CR_SS_RXN: C918.2
- new net CR_SS_RXP: C917.2
- new net CR_SS_TXN: U901.10 (RXN)
- new net CR_SS_TXP: U901.11 (RXP)
- new net CR_TXN_IC: C918.1, U901.7 (TXN)
- new net CR_TXP_IC: C917.1, U901.8 (TXP)
- new net CR_USD_CDZ: J902.9 (SW_B), R905.1, U901.36 (SD2_CDZ)
- new net CR_USD_CLK: J902.5 (CLK), U901.29 (S2CK_M2D0)
- new net CR_USD_CMD: J902.3 (CMD), U901.30 (S2CM_M2D2)
- new net CR_USD_D0: J902.7 (DAT0), U901.28 (S2D0_M2D1)
- new net CR_USD_D1: J902.8 (DAT1), U901.27 (S2D1_M2BS)
- new net CR_USD_D2: J902.1 (DAT2), U901.32 (S2D2_M2CK)
- new net CR_USD_D3: J902.2 (CD/DAT3), U901.31 (S2D3_M2D3)
- new net CR_USD_VCC: C915.1, C916.1, J902.4 (VDD), U901.24 (S2M2_VCC)
- new net CR_VUHS1: C911.1, U901.43 (VUHS_1)
- new net CR_VUHS2: C912.1, U901.33 (VUHS_2)
- new net CR_XI: C919.1, U901.13 (X1), Y901.1
- new net CR_XO: C920.1, U901.14 (X2), Y901.3
- new net GND: C901.2, C902.2, C903.2, C904.2, C905.2, C906.2, C907.2, C908.2, C909.2, C910.2, C911.2, C912.2, C913.2, C914.2, C915.2, C916.2, C919.2, C920.2, D901.1 (K), J901.12 (EP), J901.13 (EP), J901.3 (VSS1), J901.6 (VSS2), J902.10, J902.11 (SW_A), J902.12, J902.13, J902.14, J902.6 (VSS), R901.2, R903.2, U901.12 (GND), U901.3 (GND), U901.35 (MS2_INS/SD2_WP), U901.49 (EP), Y901.2 (G), Y901.4 (G)
- no-connect marks 0 -> 6
Other:
- note added: "1. GL3224-ONY04 USB 3.1 Gen1 (5 Gbps) 2-LUN card reader, QFN-48 7x7, EP = GND (via array)"
- note added: "2. POWER +5V -> VBUS; internal LDOs -> CR_3V3 (pin 25), CR_1V2 (pin 26)"
- note added: "3. USB / CLOCK / RTERM / ROM OPTIONS"
- note added: "4. CARD SOCKETS slot 1 = full-size SD (S1*), slot 2 = microSD (S2*). Both push-push."
- note added: "5. CARD DETECT / ACTIVITY -> RP2350 (read-only)"
- note added: "50 Ohm group, length-matched +-1 mm, CLK with GND guard (SDR104 = 208 MHz), keep stubs to zero."
- note added: "Budget: GL3224 147 mA (SS U0 active) + up to ~200 mA per UHS-I card, all through the internal 5->3.3 V LDO:"
- note added: "CMD / DAT0-3 pull-ups: GL3224 internal 15k (DS table 5.3) -> no external resistors. Route each slot's CLK/CMD/DAT as a"
- note added: "CR_LED: GL3224 LED output (push-pull 3.3 V, active high = access), 1k to the RP2350 GPIO (firmware shows activity on the LCD)."
- note added: "Crystal: GL3224 accepts 25 MHz +-0.03 %; same YXC 3225 part as the hub (JLC basic)."
- note added: "DM3AT: normally-open detect switch SW_A (GND) - SW_B (CDZ). microSD has no WP -> SD2_WP strapped low (write enabled)."
- note added: "DVDD12 1 uF, VUHS 0.1-1 uF, card VCC up to 10 uF. Card power is switched by the GL3224's on-chip FETs (S1M1_VCC / S2M2_VCC);"
- note added: "GL3224 is USB 3.1 Gen1: hub port 1 trains at 5 Gbps (~400 MB/s) - well above UHS-I SDR104 (104 MB/s)."
- note added: "Gen1 transmitter AC cap range is 75-200 nF, so 100 nF here (the 220 nF Gen2 value is out of range for a Gen1 TX)."
- note added: "Genesys GL3224(E) demo board V3.00 + open GL3224 designs: VBUS 2.2-10 uF, DVDD33 2.2-10 uF, AVDD33/DVDD33 pins 0.1-1 uF, AVDD12 2.2 uF,"
- note added: "Hub link: CR_SS_TX* = hub transmits (220 nF on usb_hub) -> GL3224 RXP/RXN direct. GL3224 TXP/TXN -> 100 nF here -> CR_SS_RX* -> hub."
- note added: "No reset pin: internal POR. Boots from ROM (no SPI flash). SPI_CS / SPI_MOSI NC, S1D4-7 NC (MMC 8-bit only)."
- note added: "Pin 2 is MS1_INS/SD1_WP: with no card the WP switch is open (high) so no false Memory Stick insert is seen."
- note added: "SD-111 (Hanbo drawing): CD switch to pin 3 VSS1 closes with a card; WP switch to GND closes when the card is UNLOCKED, open when"
- note added: "The GL3224 needs the card-detect switches itself (SD1_CDZ / SD2_CDZ, 46k internal pull-up to CR_3V3, low = card)."
- note added: "The RP2350 taps the same nodes through 1k: input only, internal pulls OFF (a ~50k MCU pull-down would form a divider"
- note added: "VBUS = +5V (4.75-5.25 V). CR_3V3 / CR_1V2 are the GL3224's own LDO outputs: never tie them to +3V3 or any other rail."
- note added: "card VCC kept at 4.7 uF + 100 nF so the internal 3.3 V LDO is not dipped at card power-on (proven designs use up to 10 uF)."
- note added: "derived from +5V, so the MCU never sees the node while unpowered in a way that back-feeds the GL3224."
- note added: "locked or no card -> GL3224 SD1_WP (46k internal pull-up): 0 = write enable, 1 = write protect. Matches directly, no inverter."
- note added: "with the 46k pull-up). 1k limits current if the GPIO is ever driven. CR_3V3 exists whenever +5V does, and +3V3 is"
- note added: "~(5.1-3.3) V x 0.35 A = 0.63 W in the QFN (theta-JA 33 C/W -> +21 K). Thermal pad via array to inner GND planes."
- note removed: "TODO — planned contents: Genesys GL3224-ONY04 (2 LUN), Hanbo SD-111 SD socket, Hirose DM3AT microSD, card detect -> RP2350."
- title: odeck-10 — Card reader -> odeck-10 — SD / microSD card reader (GL3224)

Commit message: Schematic review + footprint verification; fix all MAJOR findings
Reviews (docs/review/): power, PD/mux, data path, MCU/UI - 0 blockers,
7 majors, all resolved:
- power: diode-OR inputs (no shutdown-based PD-in priority), sink hand-over
  gated by delayed PG_5V, PD-in capacitance within 100 uF, HV resistor sizes,
  OVP filter/threshold, VBB_PG soft-start qualification
- card reader MS2_INS/SD2_WP phantom card, hub VBUS_DET level buffer
- RP2350 inductor dot text; minors across all sheets (HPD pull-down, PMG1
  INT pin, PHY TX caps, erratum E9 pull-downs, PHY I2C bridge gating,
  backlight 39 ohm, +1V1 cap, IOX P7)
Footprints: all 54 custom footprints checked vs manufacturer drawings,
50 fixed (courtyards, pads, paste, RJ45 mirrored pinout, EP sizes, holes);
removed obsolete FL_001 placeholder.
Firmware rules collected in docs/design/mcu.md.
186 parts, all JLC stock >= 5; netlist verify OK; ERC clean.

Co-Authored-By: Claude Opus 5.5 <noreply@anthropic.com>
Connections:
- net CR_USD_CDZ: now also U901.35 (MS2_INS/SD2_WP)
- net GND: no longer U901.35 (MS2_INS/SD2_WP)
Other:
- note added: "(same state as slot 1 with an unlocked SD). Two 46k internal pull-ups in parallel on the node (~23k) - fine."
- note added: "1k limits current if the pin is ever mis-configured as output. CR_3V3 exists whenever +5V does, and +3V3 is derived"
- note added: "5. CARD DETECT -> TCA9534 P3/P4, ACTIVITY -> RP2350 (read-only)"
- note added: "Bench item: the ROM must give SDx_CDZ = 0 priority over MSx_INS = 0 (DS silent) - unlocked SD in each slot enumerates"
- note added: "CR_USD_CDZ also drives GL3224 pin 35 (MS2_INS/SD2_WP), see section 4."
- note added: "DM3AT: normally-open detect switch SW_A (GND) - SW_B (CDZ). Pin 35 MS2_INS/SD2_WP is tied to CR_USD_CDZ (NOT GND): it is also"
- note added: "The TCA9534 (mcu, P3/P4) taps the same nodes through 1k: input only, no internal pulls (TCA9534 DS 8), 5 V tolerant."
- note added: "as writable SD, not MS. If not: inverter/strap, ask Genesys FAE."
- note added: "from +5V, so the expander never sees the node while unpowered in a way that back-feeds the GL3224."
- note added: "the Memory Stick insert input (0 = MS inserted). No card: CDZ high -> no MS, no WP. Card: low -> SD present, write enabled"
- note removed: "5. CARD DETECT / ACTIVITY -> RP2350 (read-only)"
- note removed: "DM3AT: normally-open detect switch SW_A (GND) - SW_B (CDZ). microSD has no WP -> SD2_WP strapped low (write enabled)."
- note removed: "The RP2350 taps the same nodes through 1k: input only, internal pulls OFF (a ~50k MCU pull-down would form a divider"
- note removed: "derived from +5V, so the MCU never sees the node while unpowered in a way that back-feeds the GL3224."
- note removed: "with the 46k pull-up). 1k limits current if the GPIO is ever driven. CR_3V3 exists whenever +5V does, and +3V3 is"

Commit message: Cost pass, PCB sync + rough placement, renders, README
- cost pass: extended parts 129 -> 114 (~$45/order less), nets unchanged
- tools/pcbsync.py: scripted update-PCB-from-schematic (keeps placed parts)
- tools/set_outline.py; board grown to 130x85 mm (provisional)
- hardware/odeck-10/placement.py: edge connectors + anchor-based packing,
  small passives spill to bottom; all 796 parts on the board (2 at anchor)
- docs/images: top/bottom/iso renders of the rough placement
- README.md: overview, architecture, repo layout, workflow, roadmap

Co-Authored-By: Claude Opus 5.5 <noreply@anthropic.com>
Parts:
- R901: footprint Resistor_SMD:R_0402_1005Metric -> Resistor_SMD:R_0603_1608Metric; LCSC C137948 -> C23228
Changed lines of the file:
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@@
 			)
 		)
-		(property "Footprint" "Resistor_SMD:R_0402_1005Metric"
+		(property "Footprint" "Resistor_SMD:R_0603_1608Metric"
 			(at 223.52 40.64 0)
 			(effects
@@
 			)
 		)
-		(property "LCSC" "C137948"
+		(property "LCSC" "C23228"
 			(at 223.52 40.64 0)
 			(effects

Commit message: Placement: floorplan, per-region placement scripts, DRC-clean placed board
- docs/floorplan.md: 5 regions; board 130x89 mm (SD socket depth), microSD on
  top at the front-right (overhangs edge 2 mm under the LCD panel)
- layout/{power,usbc,hubrails,front,right}.py + zz_integration.py; per-block
  placement rationale and routing intent in docs/layout-notes/
- tools/apply_layout.py (region/ownership/overlap checks), set_outline.py,
  pcbsync --refresh, apply_routing.py (coupled pairs, via pairs, zones),
  autoroute.py (Freerouting 2.4, headless, analytics off)
- schematic: R908 22R microSD CLK series termination
- footprints: PMG1 closed courtyard, barrel peg NPTH
- DRC rules (.kicad_dru): edge parts, HS pair spacing, HV clearance;
  HS netclass pad clearance 0.15
- DRC: 0 violations (499 unrouted, as expected); renders updated

Co-Authored-By: Claude Opus 5.5 <noreply@anthropic.com>
Parts:
- added R908: 22, Resistor_SMD:R_0402_1005Metric, symbol Device:R
Connections:
- net CR_USD_CLK: now also R908.1; no longer J902.5 (CLK)
- new net CR_USD_CLK_S: J902.5 (CLK), R908.2
Changed lines of the file:
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@@
 		)
 	)
-	(label "CR_USD_CLK"
+	(label "CR_USD_CLK_S"
 		(at 265.43 148.59 180)
 		(effects
@@
 		)
 	)
+	(symbol
+		(lib_id "Device:R")
+		(at 20.32 30.48 0)
+		(unit 1)
+		(exclude_from_sim no)
+		(in_bom yes)
+		(on_board yes)
+		(dnp no)
+		(property "Reference" "R908"
+			(at 22.86 29.21 0)
+			(effects
+				(font
+					(size 1.27 1.27)
+				)
+			)
+		)
+		(property "Value" "22"
+			(at 22.86 31.75 0)
+			(effects
+				(font
+					(size 1.27 1.27)
+				)
+			)
+		)
+		(property "Footprint" "Resistor_SMD:R_0402_1005Metric"
+			(at 20.32 30.48 0)
+			(effects
+				(font
+					(size 1.27 1.27)
+				)
+				(hide yes)
+			)
+		)
+		(property "Datasheet" ""
+			(at 20.32 30.48 0)
+			(effects
+				(font
+					(size 1.27 1.27)
+				)
+				(hide yes)
+			)
+		)
+		(property "Description" "microSD CLK source series termination, at the GL3224 pin (tune 22-33 R on the bench)"
+			(at 20.32 30.48 0)
+			(effects
+				(font
+					(size 1.27 1.27)
+				)
+				(hide yes)
+			)
+		)
+		(property "LCSC" "C25092"
+			(at 20.32 30.48 0)
+			(effects
+				(font
+					(size 1.27 1.27)
+				)
+				(hide yes)
+			)
+		)
+		(pin "1"
+		)
+		(pin "2"
+		)
+		(instances
+			(project "odeck-10"
+				(path "/ab49eecb-8bd6-4c6e-bedf-bbb6873dcd24/8054b97d-7891-41ee-a434-075092ac292a"
+					(reference "R908")
+					(unit 1)
+				)
+			)
+		)
+	)
+	(wire
+		(pts
+			(xy 20.32 26.67) (xy 20.32 24.13)
+		)
+		(stroke
+			(width 0)
+			(type default)
+		)
+	)
+	(label "CR_USD_CLK"
+		(at 20.32 24.13 90)
+		(effects
+			(font
+				(size 1.27 1.27)
+			)
+			(justify left bottom)
+		)
+	)
+	(wire
+		(pts
+			(xy 20.32 34.29) (xy 20.32 36.83)
+		)
+		(stroke
+			(width 0)
+			(type default)
+		)
+	)
+	(label "CR_USD_CLK_S"
+		(at 20.32 36.83 270)
+		(effects
+			(font
+				(size 1.27 1.27)
+			)
+			(justify right bottom)
+		)
+	)
